File: EAGLE Board Designs/BMS/BMS Segment/BMS Segment rev15 new.brd (EAGLE design)
At the start: 108 x 240.3 mm, 294 parts, among them J1_A 0R, J1_B 0R, J2_A 0R, J2_B 0R, J3_A 0R, J3_B 0R, J4_A 0R, J4_B 0R, J5_A 0R, J5_B 0R, J6_A 0R, J6_B 0R, J7_A 0R, J7_B 0R, J8_A 0R, J8_B 0R, Q1 NSV1C201MZ4, Q2 NSV1C201MZ4, U1 LTC6811-2, U2 LTC6811-2

Commit message: Started changing the silkscreen to have reference indicators
Parts:
- renumbered DRAIN10:C to DC10:C1, DRAIN10:DISCHARGE to DC10:R3, DRAIN10:GATE to DC10:R2, DRAIN10:LED1 to DC10:D1, DRAIN10:PFET to DC10:PFET, DRAIN10:R to DC10:R1, DRAIN10:R1 to DC10:R4, DRAIN11:C to DC11:C1, DRAIN11:DISCHARGE to DC11:R3, DRAIN11:GATE to DC11:R2, DRAIN11:LED1 to DC11:D1, DRAIN11:PFET to DC11:PFET, DRAIN11:R to DC11:R1, DRAIN11:R1 to DC11:R4, DRAIN12:C to DC12:C1, DRAIN12:DISCHARGE to DC12:R3, DRAIN12:GATE to DC12:R2, DRAIN12:LED1 to DC12:D1, DRAIN12:PFET to DC12:PFET, DRAIN12:R to DC12:R1, DRAIN12:R1 to DC12:R4, DRAIN13:C to DC13:C1, DRAIN13:DISCHARGE to DC13:R3, DRAIN13:GATE to DC13:R2, DRAIN13:LED1 to DC13:D1, DRAIN13:PFET to DC13:PFET, DRAIN13:R to DC13:R1, DRAIN13:R1 to DC13:R4, DRAIN14:C to DC14:C1, DRAIN14:DISCHARGE to DC14:R3, DRAIN14:GATE to DC14:R2, DRAIN14:LED1 to DC14:D1, DRAIN14:PFET to DC14:PFET, DRAIN14:R to DC14:R1, DRAIN14:R1 to DC14:R4, DRAIN15:C to DC15:C1, DRAIN15:DISCHARGE to DC15:R3, DRAIN15:GATE to DC15:R2, DRAIN15:LED1 to DC15:D1, DRAIN15:PFET to DC15:PFET, DRAIN15:R to DC15:R1, DRAIN15:R1 to DC15:R4, DRAIN16:C to DC16:C1, DRAIN16:DISCHARGE to DC16:R3, DRAIN16:GATE to DC16:R2, DRAIN16:LED1 to DC16:D1, DRAIN16:PFET to DC16:PFET, DRAIN16:R to DC16:R1, DRAIN16:R1 to DC16:R4, DRAIN17:C to DC17:C1, DRAIN17:DISCHARGE to DC17:R3, DRAIN17:GATE to DC17:R2, DRAIN17:LED1 to DC17:D1, DRAIN17:PFET to DC17:PFET, DRAIN17:R to DC17:R1, DRAIN17:R1 to DC17:R4, DRAIN18:C to DC18:C1, DRAIN18:DISCHARGE to DC18:R3, DRAIN18:GATE to DC18:R2, DRAIN18:LED1 to DC18:D1, DRAIN18:PFET to DC18:PFET, DRAIN18:R to DC18:R1, DRAIN18:R1 to DC18:R4, DRAIN1:C to DC1:C1, DRAIN1:DISCHARGE to DC1:R3, DRAIN1:GATE to DC1:R2, DRAIN1:LED1 to DC1:D1, DRAIN1:PFET to DC1:PFET, DRAIN1:R to DC1:R1, DRAIN1:R1 to DC1:R4, DRAIN2:C to DC2:C1, DRAIN2:DISCHARGE to DC2:R3, DRAIN2:GATE to DC2:R2, DRAIN2:LED1 to DC2:D1, DRAIN2:PFET to DC2:PFET, DRAIN2:R to DC2:R1, DRAIN2:R1 to DC2:R4, DRAIN3:C to DC3:C1, DRAIN3:DISCHARGE to DC3:R3, DRAIN3:GATE to DC3:R2, DRAIN3:LED1 to DC3:D1, DRAIN3:PFET to DC3:PFET, DRAIN3:R to DC3:R1, DRAIN3:R1 to DC3:R4, DRAIN4:C to DC4:C1, DRAIN4:DISCHARGE to DC4:R3, DRAIN4:GATE to DC4:R2, DRAIN4:LED1 to DC4:D1, DRAIN4:PFET to DC4:PFET, DRAIN4:R to DC4:R1, DRAIN4:R1 to DC4:R4, DRAIN5:C to DC5:C1, DRAIN5:DISCHARGE to DC5:R3, DRAIN5:GATE to DC5:R2, DRAIN5:LED1 to DC5:D1, DRAIN5:PFET to DC5:PFET, DRAIN5:R to DC5:R1, DRAIN5:R1 to DC5:R4, DRAIN6:C to DC6:C1, DRAIN6:DISCHARGE to DC6:R3, DRAIN6:GATE to DC6:R2, DRAIN6:LED1 to DC6:D1, DRAIN6:PFET to DC6:PFET, DRAIN6:R to DC6:R1, DRAIN6:R1 to DC6:R4, DRAIN7:C to DC7:C1, DRAIN7:DISCHARGE to DC7:R3, DRAIN7:GATE to DC7:R2, DRAIN7:LED1 to DC7:D1, DRAIN7:PFET to DC7:PFET, DRAIN7:R to DC7:R1, DRAIN7:R1 to DC7:R4, DRAIN8:C to DC8:C1, DRAIN8:DISCHARGE to DC8:R3, DRAIN8:GATE to DC8:R2, DRAIN8:LED1 to DC8:D1, DRAIN8:PFET to DC8:PFET, DRAIN8:R to DC8:R1, DRAIN8:R1 to DC8:R4, DRAIN9:C to DC9:C1, DRAIN9:DISCHARGE to DC9:R3, DRAIN9:GATE to DC9:R2, DRAIN9:LED1 to DC9:D1, DRAIN9:PFET to DC9:PFET, DRAIN9:R to DC9:R1, DRAIN9:R1 to DC9:R4, THERM_FILTER10:C to T_FIL10:C1, THERM_FILTER10:R to T_FIL10:R2, THERM_FILTER10:R1 to T_FIL10:R1, THERM_FILTER1:C to T_FIL1:C1, THERM_FILTER1:R to T_FIL1:R2, THERM_FILTER1:R1 to T_FIL1:R1, THERM_FILTER2:C to T_FIL2:C1, THERM_FILTER2:R to T_FIL2:R2, THERM_FILTER2:R1 to T_FIL2:R1, THERM_FILTER3:C to T_FIL3:C1, THERM_FILTER3:R to T_FIL3:R2, THERM_FILTER3:R1 to T_FIL3:R1, THERM_FILTER4:C to T_FIL4:C1, THERM_FILTER4:R to T_FIL4:R2, THERM_FILTER4:R1 to T_FIL4:R1, THERM_FILTER5:C to T_FIL5:C1, THERM_FILTER5:R to T_FIL5:R2, THERM_FILTER5:R1 to T_FIL5:R1, THERM_FILTER6:C to T_FIL6:C1, THERM_FILTER6:R to T_FIL6:R2, THERM_FILTER6:R1 to T_FIL6:R1, THERM_FILTER7:C to T_FIL7:C1, THERM_FILTER7:R to T_FIL7:R2, THERM_FILTER7:R1 to T_FIL7:R1, THERM_FILTER8:C to T_FIL8:C1, THERM_FILTER8:R to T_FIL8:R2, THERM_FILTER8:R1 to T_FIL8:R1, THERM_FILTER9:C to T_FIL9:C1, THERM_FILTER9:R to T_FIL9:R2, THERM_FILTER9:R1 to T_FIL9:R1
Connections:
- net DRAIN10:GATE renamed DC10:GATE
- net DRAIN10:N$1 renamed DC10:N$1
- net DRAIN10:N$2 renamed DC10:N$2
- net DRAIN11:GATE renamed DC11:GATE
- net DRAIN11:N$1 renamed DC11:N$1
- net DRAIN11:N$2 renamed DC11:N$2
- net DRAIN12:GATE renamed DC12:GATE
- net DRAIN12:N$1 renamed DC12:N$1
- net DRAIN12:N$2 renamed DC12:N$2
- net DRAIN13:GATE renamed DC13:GATE
- net DRAIN13:N$1 renamed DC13:N$1
- net DRAIN13:N$2 renamed DC13:N$2
- net DRAIN14:GATE renamed DC14:GATE
- net DRAIN14:N$1 renamed DC14:N$1
- net DRAIN14:N$2 renamed DC14:N$2
- net DRAIN15:GATE renamed DC15:GATE
- net DRAIN15:N$1 renamed DC15:N$1
- net DRAIN15:N$2 renamed DC15:N$2
- net DRAIN16:GATE renamed DC16:GATE
- net DRAIN16:N$1 renamed DC16:N$1
- net DRAIN16:N$2 renamed DC16:N$2
- net DRAIN17:GATE renamed DC17:GATE
- net DRAIN17:N$1 renamed DC17:N$1
- net DRAIN17:N$2 renamed DC17:N$2
- net DRAIN18:GATE renamed DC18:GATE
- net DRAIN18:N$1 renamed DC18:N$1
- net DRAIN18:N$2 renamed DC18:N$2
- net DRAIN1:GATE renamed DC1:GATE
- net DRAIN1:N$1 renamed DC1:N$1
- net DRAIN1:N$2 renamed DC1:N$2
- net DRAIN2:GATE renamed DC2:GATE
- net DRAIN2:N$1 renamed DC2:N$1
- net DRAIN2:N$2 renamed DC2:N$2
- net DRAIN3:GATE renamed DC3:GATE
- net DRAIN3:N$1 renamed DC3:N$1
- net DRAIN3:N$2 renamed DC3:N$2
- net DRAIN4:GATE renamed DC4:GATE
- net DRAIN4:N$1 renamed DC4:N$1
- net DRAIN4:N$2 renamed DC4:N$2
- net DRAIN5:GATE renamed DC5:GATE
- net DRAIN5:N$1 renamed DC5:N$1
- net DRAIN5:N$2 renamed DC5:N$2
- net DRAIN6:GATE renamed DC6:GATE
- net DRAIN6:N$1 renamed DC6:N$1
- net DRAIN6:N$2 renamed DC6:N$2
- net DRAIN7:GATE renamed DC7:GATE
- net DRAIN7:N$1 renamed DC7:N$1
- net DRAIN7:N$2 renamed DC7:N$2
- net DRAIN8:GATE renamed DC8:GATE
- net DRAIN8:N$1 renamed DC8:N$1
- net DRAIN8:N$2 renamed DC8:N$2
- net DRAIN9:GATE renamed DC9:GATE
- net DRAIN9:N$1 renamed DC9:N$1
- net DRAIN9:N$2 renamed DC9:N$2

Commit message: Fixed silkscreen for ref ind, switched pogos for springs, altered traces
Parts:
- CELL0, CELL1, CELL10, CELL11, CELL12, CELL13, CELL14, CELL15, CELL16, CELL17, CELL18, CELL2, CELL3, CELL4, CELL5, CELL6, CELL7, CELL8, CELL9: value BATTERY_SPRING_SPRING_CONTACT -> BATTERY_SPRING_KEYSTONE5222; device HyTechDevices:CONTACT_SPRING -> HyTechDevices - Copy:KEYSTONE5222
Connections:
- net CC0: now also CELL0.1; no longer CELL0.P$1
- net CC1: now also CELL1.1; no longer CELL1.P$1
- net CC10: now also CELL10.1; no longer CELL10.P$1
- net CC11: now also CELL11.1; no longer CELL11.P$1
- net CC12: now also CELL12.1; no longer CELL12.P$1
- net CC13: now also CELL13.1; no longer CELL13.P$1
- net CC14: now also CELL14.1; no longer CELL14.P$1
- net CC15: now also CELL15.1; no longer CELL15.P$1
- net CC16: now also CELL16.1; no longer CELL16.P$1
- net CC17: now also CELL17.1; no longer CELL17.P$1
- net CC18: now also CELL18.1; no longer CELL18.P$1
- net CC2: now also CELL2.1; no longer CELL2.P$1
- net CC3: now also CELL3.1; no longer CELL3.P$1
- net CC4: now also CELL4.1; no longer CELL4.P$1
- net CC5: now also CELL5.1; no longer CELL5.P$1
- net CC6: now also CELL6.1; no longer CELL6.P$1
- net CC7: now also CELL7.1; no longer CELL7.P$1
- net CC8: now also CELL8.1; no longer CELL8.P$1
- net CC9: now also CELL9.1; no longer CELL9.P$1
Routing:
- net SENSE18: track 155.8 -> 163.0 mm
- net DC4:N$1: track 12.3 -> 16.9 mm
- net CC1: track 10.6 -> 14.2 mm
- net SENSE17_POST: track 118.5 -> 120.5 mm
- net V-_A: track 824.4 -> 826.3 mm
- net S3_B: track 120.0 -> 118.7 mm
- net CC5: vias 1 -> 2
- net CC3: vias 1 -> 2
- net CC2: vias 1 -> 2
- net CC18: vias 1 -> 2
- net CC17: vias 1 -> 2
- net CC13: vias 1 -> 2

Commit message: Finished fixing silkscreen and adding names
Parts:
- renumbered DC10:PFET to DC10:Q1, DC11:PFET to DC11:Q1, DC12:PFET to DC12:Q1, DC13:PFET to DC13:Q1, DC14:PFET to DC14:Q1, DC15:PFET to DC15:Q1, DC16:PFET to DC16:Q1, DC17:PFET to DC17:Q1, DC18:PFET to DC18:Q1, DC1:PFET to DC1:Q1, DC2:PFET to DC2:Q1, DC3:PFET to DC3:Q1, DC4:PFET to DC4:Q1, DC5:PFET to DC5:Q1, DC6:PFET to DC6:Q1, DC7:PFET to DC7:Q1, DC8:PFET to DC8:Q1, DC9:PFET to DC9:Q1, TRANSFORMER to T1
Routing:
- net CC4: track 24.9 -> 15.6 mm
- net CC2: track 28.6 -> 26.3 mm
- net CC15: track 21.3 -> 19.3 mm
- net SENSE7: track 66.6 -> 64.7 mm
- net SENSE13: track 65.7 -> 64.0 mm
- net SENSE1: track 80.3 -> 78.6 mm
- net DC2:N$1: track 17.4 -> 16.5 mm
- net DC7:N$1: track 14.2 -> 13.4 mm
- net DC10:N$1: track 20.2 -> 19.5 mm
- net DC18:N$1: track 19.3 -> 18.6 mm
- net DC5:N$1: track 14.2 -> 13.6 mm
- net SENSE12: track 59.5 -> 60.1 mm
- net DC13:N$1: track 14.0 -> 14.6 mm
Other:
- board text added: "T1"
- board text added: "U1"
- board text added: "U2"
