File: EAGLE Board Designs/BMS/BMS Segment/BMS Segment rev15.sch (EAGLE design)
At the start: 73 parts, among them J0 CONNECTOR-1, J1 CONNECTOR-1, J10 CONNECTOR-1, J11 CONNECTOR-1, J12 CONNECTOR-1, J13 CONNECTOR-1, J14 CONNECTOR-1, J15 CONNECTOR-1, J16 CONNECTOR-1, J17 CONNECTOR-1, J18 CONNECTOR-1, J2 CONNECTOR-1, J3 CONNECTOR-1, J4 CONNECTOR-1, J5 CONNECTOR-1, J6 CONNECTOR-1, J7 CONNECTOR-1, J8 CONNECTOR-1, J9 CONNECTOR-1, T1 TRANSFORMER, U1 LTC6813

Commit message: Final BMS rev15 design
Parts:
- removed C1, C2, C3: CAPACITOR_0603_10V_1UF, HyTechDevices:CAPACITOR_0603_10V_1UF
- removed C5, C6, C7, C8: CAPACITOR_0603_10V_10NF, HyTechDevices:CAPACITOR_0603_10V_10NF
- removed CELL0.C1: CAPACITOR_0603_100V_10NF, HyTechDevices:CAPACITOR_0603_100V_10NF
- removed CELL0.R1, DRIVE.R1, SENSE18.R1: RESISTOR_0603_100, HyTechDevices:RESISTOR_0603_100
- removed DRIVE.C1, SENSE18.C1: CAPACITOR_0603_100V_0.1UF, HyTechDevices:CAPACITOR_0603_100V_0.1UF
- removed J0, J1, J10, J11, J12, J13, J14, J15, J16, J17, J18, J2, J3, J4, J5, J6, J7, J8, J9: CONNECTOR-1, HyTechDevices:CONNECTOR-1
- removed J19, J20, J21, J22, J23, J24, J26: (no value), HyTechDevices:CONNECTOR-2_NANOFIT_SMD_VERTICAL_BLACK
- removed J25: (no value), HyTechDevices:CONNECTOR-2_NANOFIT_SMD_VERTICAL_NATURAL
- removed J27, J28: (no value), HyTechDevices:JUMPER_NANOFIT_SMD_VERTICAL_NATURAL
- removed R1, R2: RESISTOR_0603_1K, HyTechDevices:RESISTOR_0603_1K
- removed R3, R4, R5, R6: RESISTOR_0603_60.4, HyTechDevices:RESISTOR_0603_60.4
- removed RT1, RT2, RT3: THERMISTOR, HyTechDevices:THERMISTOR
- added C1_A, C1_B, C2_A, C2_B, C8_A, C8_B: 1uF, HyTechDevices:CAP0603-CAP
- added C3_A, C3_B: 15pF, HyTechDevices:CAP0603-CAP
- added C4_A, C4_B, C5_A, C_5: 10nF, HyTechDevices:CAP0603-CAP
- added C6_A, C6_B, C7_A, C7_B: 100nF, HyTechDevices:CAP0603-CAP
- added CELL0, CELL1, CELL10, CELL11, CELL12, CELL13, CELL14, CELL15, CELL16, CELL17, CELL18, CELL2, CELL3, CELL4, CELL5, CELL6, CELL7, CELL8, CELL9: BATTERY_SPRING_KEYSTONE5222, HyTechDevices - Copy:BATTERY_SPRING_KEYSTONE5222
- added ISOSPI_A, ISOSPI_B: ISOSPI, HyTechDevices:CONNECTOR-2NANO-FIT_VERTICAL-2
- added J1_A, J1_B, J2_A, J2_B, J3_A, J3_B, J4_A, J4_B, J5_A, J5_B, J6_A, J6_B, J7_A, J7_B, J8_A, J8_B, J_CELL_A, J_THERM_A: 0R, HyTechDevices:RESISTOR0603-RES
- added Q2: NSV1C201MZ4, HyTechDevices:NSV1C201MZ4
- added R1_A, R1_B, R2_A, R2_B, RIN_A, RIN_B, RM_A, RM_B, RU1_A, RU1_B, RU2_A, RU2_B: 100R, HyTechDevices:RESISTOR0603-RES
- added R3_A, R3_B: 402R, HyTechDevices:RESISTOR0603-RES
- added R4_A, R4_B, R5_A, R5_B: 22R, HyTechDevices:RESISTOR0603-RES
- added RB1_A, RB1_B: 1K2, HyTechDevices:RESISTOR0603-RES
- added RB2_A, RB2_B: 806R, HyTechDevices:RESISTOR0603-RES
- added THERM1, THERM2, THERM3, THERM4: 10K, HyTechDevices:THERMISTOR_NCP210603
- added THERM1_A, THERM1_B, THERM2_A, THERM2_B, THERM3_A, THERM3_B: THERMISTOR, HyTechDevices:CONNECTOR-2NANO-FIT_VERTICAL-2
- added TP1, TP2, TP3, TP4, TP5, TP6: TEST_POINTMICRO_MINIATURE, HyTechDevices - Copy:TEST_POINTMICRO_MINIATURE
- added U2: LTC6811-2, HyTechDevices:LTC6811-2
- F0, F1, F10, F11, F12, F13, F14, F15, F16, F17, F18, F2, F3, F4, F5, F6, F7, F8, F9: value (none) -> 0001.2704.11; RATING (none) -> 1A
- Q1: value (none) -> NSV1C201MZ4; device HyTechDevices:TRANSISTOR_NPN -> HyTechDevices:NSV1C201MZ4
- T1: value TRANSFORMER -> HM2102NLT; device HyTechDevices:TRANSFORMER -> HyTechDevices:HM2102NLT
- U1: value LTC6813 -> LTC6811-2; device HyTechDevices:LTC6813 -> HyTechDevices:LTC6811-2
Connections:
- net C1 renamed C1_A
- net C10 renamed C10_A
- net C2 renamed C2_A
- net C3 renamed C3_A
- net C4 renamed C4_A
- net C5 renamed C5_A
- net C7 renamed C7_A
- net C8 renamed C8_A
- net C9 renamed C9_A
- net GPIO2 renamed GPIO2_A
- net GPIO4 renamed GPIO4_A
- net GPIO5 renamed GPIO5_A
- net S1 renamed S1_A
- net S10 renamed S10_A
- net S2 renamed S2_A
- net S3 renamed S3_A
- net S4 renamed S4_A
- net S5 renamed S5_A
- net S7 renamed S7_A
- net S8 renamed S8_A
- net S9 renamed S9_A
- removed net C(N): C1.1, R1.2
- removed net C0: CELL0.C1.1, CELL0.R1.2, U1.C0
- removed net C11: U1.C11
- removed net C12: U1.C12
- removed net C13: U1.C13
- removed net C14: U1.C14
- removed net C15: U1.C15
- removed net C16: U1.C16
- removed net C17: U1.C17
- removed net C18: U1.C18
- removed net C6: U1.C6
- removed net CELL-: R3.1, R4.1
- removed net DRIVE: Q1.BASE, U1.DRIVE
- removed net GPIO: C1.1, R1.1
- removed net GPIO1: J27.P$1, U1.GPI01
- removed net GPIO1_PRE: J27.P$2
- removed net GPIO3: U1.GPI03
- removed net GPIO6: U1.GPI06
- removed net GPIO7: U1.GPI07
- removed net GPIO8: U1.GPI08
- removed net GPIO9: U1.GPI09
- removed net IBIAS: R1.2, U1.IBIAS
- removed net ICMP: R1.1, R2.2, U1.ICMP
- removed net IMA: R3.1, T1A.TD+, U1.IMA
- removed net IMB: R5.2, T1B.TD+, U1.IMB
- removed net IPA: R4.2, T1A.TD-, U1.IPA
- removed net IPB: R6.2, T1B.TD-, U1.IPB
- removed net ISO_IMA: J25.2, T1A.MX+
- removed net ISO_IMB: J26.2, T1B.MX+
- removed net ISO_IPA: J25.1, T1A.MX-
- removed net ISO_IPB: J26.1, T1B.MX-
- removed net N$15: DRIVE.C1.1, DRIVE.R1.2, Q1.COLLECTOR
- removed net S(N): R2.2
- removed net S11: U1.S11
- removed net S12: U1.S12
- removed net S13: U1.S13
- removed net S14: U1.S14
- removed net S15: U1.S15
- removed net S16: U1.S16
- removed net S17: U1.S17
- removed net S18: U1.S18
- removed net S6: U1.S6
- removed net SENSE17: J28.P$2
- removed net SENSE17_PRE: F17.2, J28.P$1
- removed net SENSE9: F9.2
- removed net THERM: R1.2, R2.1
- removed net THERM1: J19.1
- removed net THERM2: J20.1
- removed net THERM3: J21.1
- removed net THERM4: J22.1
- removed net THERM5: J23.1
- removed net THERM6: J24.1
- removed net THERM7: RT1.2
- removed net THERM8: RT2.2
- removed net THERM9: RT3.2
- removed net V+: SENSE18.C1.1, SENSE18.R1.1, U1.V+
- removed net V-: C1.2, C2.2, C3.2, C5.2, C6.1, C7.1, C8.2, CELL0.C1.2, CELL0.R1.1, DRIVE.C1.2, F0.2, J19.2, J20.2, J21.2, J22.2, J23.2, J24.2, R2.1, RT1.1, RT2.1, RT3.1, SENSE18.C1.2, U1.V-
- removed net VREF1: C2.1, U1.VREF1
- removed net VREF2: C1.1, R2.2, U1.VREF2
- removed net VREG: C3.1, Q1.EMITTER, U1.VREG
- new net C0_A: C5_A.1, R2_A.2, U1.C0
- new net C0_B: C_5.1, R2_B.2, U2.C0
- new net C10_B: U2.C10
- new net C1_B: U2.C1
- new net C2_B: U2.C2
- new net C3_B: U2.C3
- new net C4_B: U2.C4
- new net C5_B: U2.C5
- new net C7_B: U2.C7
- new net C8_B: U2.C8
- new net C9_B: U2.C9
- new net DRIVE_A: Q1.BASE, TP6.P$1, U1.DRIVE
- new net DRIVE_B: Q2.BASE, TP5.P$1, U2.DRIVE
- new net GATE: Q1.G
- new net GPIO1_A: U1.GPI01
- new net GPIO1_B: U2.GPI01
- new net GPIO2_B: U2.GPI02
- new net GPIO3_A_POST: J_THERM_A.1, U1.GPI03
- new net GPIO3_A_PRE: J_THERM_A.2
- new net GPIO3_B: U2.GPI03
- new net GPIO4_B: U2.GPI04
- new net GPIO5_B: U2.GPI05
- new net IM_A: C3_A.2, T1G$2.TD+, U1.CSB(IMA)
- new net IM_B: C3_B.2, T1G$1.TD+, U2.CSB(IMA)
- new net IP_A: R3_A.1, T1G$2.TD-, U1.SCK(IPA)
- new net IP_B: R3_B.1, T1G$1.TD-, U2.SCK(IPA)
- new net ISOSPI-M: ISOSPI_A-2.S, ISOSPI_B-2.S, R5_A.2, R5_B.2, RM_A.2, RM_B.2
- new net ISOSPI-P: ISOSPI_A-1.S, ISOSPI_B-1.S, R4_A.2, R4_B.2, RM_A.1, RM_B.1
- new net N$1: C4_B.1, Q1.D, T1G$1.TCT
- new net N$10: C3_B.1, R3_B.2
- new net N$13: J3_B.1, J4_B.1, U2.A1
- new net N$16: J1_B.1, J2_B.1, U2.A0
- new net N$17: THERM1.2
- new net N$19: THERM2.2
- new net N$2: RB1_B.2, U2.SDO(IBIAS)
- new net N$20: RB1_A.1, RB2_A.2, U1.SDI(ICMP)
- new net N$21: C4_A.1, T1G$2.TCT
- new net N$22: R4_A.1, T1G$2.MX-
- new net N$23: R5_A.1, T1G$2.MX+
- new net N$24: C3_A.1, R3_A.2
- new net N$26: THERM3_B-1.S
- new net N$30: J7_A.1, J8_A.1, U1.A3
- new net N$31: J5_A.1, J6_A.1, U1.A2
- new net N$32: J3_A.1, J4_A.1, U1.A1
- new net N$33: J1_A.1, J2_A.1, U1.A0
- new net N$34: THERM4.2
- new net N$35: THERM3_A-1.S
- new net N$36: THERM3.2
- new net N$37: THERM2_A-1.S
- new net N$38: THERM1_A-1.S
- new net N$44: F17.2, J_CELL_A.1
- new net N$8: J7_B.1, J8_B.1, U2.A3
- new net N$9: J5_B.1, J6_B.1, U2.A2
- new net S10_B: U2.S10
- new net S1_B: U2.S1
- new net S2_B: U2.S2
- new net S3_B: U2.S3
- new net S4_B: U2.S4
- new net S5_B: U2.S5
- new net S7_B: U2.S7
- new net S8_B: U2.S8
- new net S9_B: U2.S9
- new net SENSE17_POST: J_CELL_A.2
- new net UNUSED1_A: RU1_A.2, U1.C11, U1.C12
- new net UNUSED1_B: RU1_B.2, U2.C11, U2.C12
- new net UNUSED2_A: RU2_A.2, U1.C6
- new net UNUSED2_B: RU2_B.2, U2.C6
- new net V+_A: C6_A.1, R1_A.2, U1.V+
- new net V+_B: C6_B.1, R1_B.2, U2.V+
- new net V-_A: C1_A.2, C2_A.2, C4_A.2, C5_A.2, C6_A.2, C7_A.2, C8_A.2, F9.2, J1_A.2, J3_A.2, J5_A.2, J7_A.2, R1_B.1, R2_A.1, RB2_A.1, RIN_B.1, RU1_B.1, THERM1_A-2.S, THERM2_A-2.S, THERM3.1, THERM3_A-2.S, THERM4.1, TP2.P$1, TP3.P$1, U1.V-, U1.V-**
- new net V-_B: C1_B.2, C2_B.2, C4_B.2, C6_B.2, C7_B.2, C8_B.2, C_5.2, F0.2, J1_B.2, J3_B.2, J5_B.2, J7_B.2, R2_B.1, RB2_B.1, THERM1.1, THERM1_B-2.S, THERM2.1, THERM2_B-2.S, THERM3_B-2.S, TP4.P$1, U2.V-, U2.V-**
- new net VIN_A: C7_A.1, Q1.COLLECTOR, RIN_A.2
- new net VIN_B: C7_B.1, Q2.COLLECTOR, RIN_B.2
- new net VREF1_A: C2_A.1, U1.VREF1
- new net VREF1_B: C2_B.1, U2.VREF1
- new net VREF2_A: C1_A.1, U1.VREF2
- new net VREF2_B: C1_B.1, U2.VREF2
- new net VREG_A: C8_A.1, J2_A.2, J4_A.2, J6_A.2, J8_A.2, Q1.EMITTER, U1.ISOMD, U1.SWTEN, U1.VREG
- new net VREG_B: C8_B.1, J2_B.2, J4_B.2, J6_B.2, J8_B.2, Q2.EMITTER, U2.ISOMD, U2.SWTEN, U2.VREG
- net CC0: now also CELL0.S; no longer J0.1
- net CC1: now also CELL1.S; no longer J1.1
- net CC10: now also CELL10.S; no longer J10.1
- net CC11: now also CELL11.S; no longer J11.1
- net CC12: now also CELL12.S; no longer J12.1
- net CC13: now also CELL13.S; no longer J13.1
- net CC14: now also CELL14.S; no longer J14.1
- net CC15: now also CELL15.S; no longer J15.1
- net CC16: now also CELL16.S; no longer J16.1
- net CC17: now also CELL17.S; no longer J17.1
- net CC18: now also CELL18.S; no longer J18.1
- net CC2: now also CELL2.S; no longer J2.1
- net CC3: now also CELL3.S; no longer J3.1
- net CC4: now also CELL4.S; no longer J4.1
- net CC5: now also CELL5.S; no longer J5.1
- net CC6: now also CELL6.S; no longer J6.1
- net CC7: now also CELL7.S; no longer J7.1
- net CC8: now also CELL8.S; no longer J8.1
- net CC9: now also CELL9.S; no longer J9.1
- net CELL+: no longer R1.1
- net N$18: now also THERM2_B-1.S; no longer C8.1, R5.1, R6.1
- net N$3: now also THERM1_B-1.S; no longer C5.1, T1A.TCT
- net N$4: now also RB1_B.1, RB2_B.2, U2.SDI(ICMP); no longer C7.2, T1B.TCT
- net N$5: now also R4_B.1, T1G$1.MX-; no longer C6.2, Q1.G, R2.1, R3.2, R4.1
- net N$6: now also RB1_A.2, U1.SDO(IBIAS); no longer Q1.D, R3.2
- net N$7: now also R5_B.1, T1G$1.MX+; no longer R4.2
- net SENSE14: now also RU2_A.1
- net SENSE18: now also R1_A.1, RIN_A.1, RU1_A.1, TP1.P$1; no longer DRIVE.R1.1, SENSE18.R1.2
- net SENSE5: now also RU2_B.1
Other:
- note added: "0Ω resistors to set chip address"
- note added: "3 cell thermistors and 2 PCB thermistors per LTC6811 IC"
- note added: "Arvind Srinivasan"
- note added: "CELL 9 IS SHARED BY CIRCUIT A AND CIRCUIT B"
- note added: "Cell Input"
- note added: "Cell Thermistor Filter and Resistor Divider"
- note added: "Cell Voltage Filter and Discharge Circuit"
- note added: "Circuit A (Upper 9 Cells)"
- note added: "Circuit B (Lower 9 Cells)"
- note added: "Gate Drive"
- note added: "LTC6811-2"
- note added: "RM (TERMINATION) is only to be connected on LAST segment"
- note added: "SENSE9"
- note added: "See LTC6811 Datasheet pg.70"
- note added: "See pg. 86 for unused cells (9 cells per LTC6811 in this design)"
- note added: "V-_A / SENSE9"
- note added: "VOLTAGE TAPS"
