File: EAGLE Board Designs/Testing and Practice Boards/Keychain/Keychain rev3.sch (EAGLE design)
At the start: 10 parts, among them J1 10118192-0001LF

Commit message: Keychain rev3 complete
Parts:
- removed C1: 4.7uF, HyTechDevices:CAP0603-CAP
- removed C3: 10nF, HyTechDevices:CAP0603-CAP
- removed LED: (no value), HyTechDevices:LED-0603
- removed NA555: NA555SO-8, HyTechDevices:NA555SO-8
- removed R1: 1k, HyTechDevices:RESISTOR_0603_1K
- removed R2: 43k, HyTechDevices:RESISTOR_0603_1K
- removed R3: RESISTOR_0603_1K, HyTechDevices:RESISTOR_0603_1K
- added C2: CAPACITOR_0603_10V_4.7UF, HyTechDevices:CAPACITOR_0603_10V_4.7UF
- added C4: CAPACITOR_0603_10V_10NF, HyTechDevices:CAPACITOR_0603_10V_10NF
- added D1: LED_0603_YELLOW, HyTechDevices:LED_0603_YELLOW
- added R4: RESISTOR_0603_43K, HyTechDevices:RESISTOR_0603_43K
- added R5: RESISTOR_0603_1K, HyTechDevices:RESISTOR_0603_1K
- added R6: RESISTOR_0603_240, HyTechDevices:RESISTOR_0603_240
- added U1: NA555, HyTechDevices:NA555
Connections:
- removed net N$1: LED.A, R3.2
- removed net N$13: C3.1, NA555.5
- removed net N$2: C1.1, NA555.2, NA555.6, R2.1
- removed net N$3: NA555.7, R1.2, R2.2
- removed net RED: NA555.3, R3.1
- removed net VCC: 5V.P$1, J1.VUSB, NA555.4, NA555.8, R1.1
- new net +5V: 5V.P$1, J1.VUSB, R5.2, U1.!RESET, U1.VCC
- new net N$4: C2.1, R4.1, U1.THRESHOLD, U1.TRIGGER
- new net N$5: R4.2, R5.1, U1.DISCHARGE
- new net N$6: R6.1, U1.OUTPUT
- new net N$8: D1.A, R6.2
- new net N$9: C4.1, U1.CONTROL
- net GND: now also C2.2, C4.2, D1.C, U1.GND; no longer C1.2, C3.2, LED.C, NA555.1
Other:
- moved on the sheet: J1
