File: EAGLE Board Designs/IMU CAN Speed Converter Board/IMU CAN Speed Converter Board rev1.sch (EAGLE design)
At the start: 26 parts, among them J1 CONNECTOR-CAN_NF_S_RA_BLACK, J2 CONNECTOR-CAN_NF_S_RA_BLACK, J3 JUMPER_1X02_, J4 JUMPER_1X02_, U1 LM340, U2 TCAN1051HQV-Q1, U3 TCAN1051HQV-Q1

Commit message: Finished Design Review and Manufacturing Files
Parts:
- C11: value CAPACITOR_0603_25V_0.22UF -> CAPACITOR_0603_25V_1UF; device HyTechDevices:CAPACITOR_0603_25V_0.22UF -> HyTechDevices:CAPACITOR_0603_25V_1UF
- C2: value CAPACITOR_0603_10V_0.1UF -> CAPACITOR_0603_10V_4.7UF; device HyTechDevices:CAPACITOR_0603_10V_0.1UF -> HyTechDevices:CAPACITOR_0603_10V_4.7UF
- U1: value LM340 -> VOLTAGE_REGULATOR_SOT223_5V; device HyTechDevices:LM340 -> HyTechDevices:VOLTAGE_REGULATOR_SOT223_5V
Changed lines of the file:
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@@
 </classes>
 <parts>
-<part name="FRAME1" library="HyTechFrames" deviceset="FRAME" device=""/>
-<part name="U1" library="HyTechDevices" deviceset="LM340" device=""/>
+<part name="FRAME1" library="HyTechFrames" deviceset="FRAME" device="">
+<attribute name="DESCRIPTION_1" value="Convert IMU's CAN speed from 1Mbps to 500 kbps"/>
+<attribute name="DESIGNER_SCHEMATIC" value="Bo Han Zhu"/>
+<attribute name="ENGINEER" value="Bo Han Zhu"/>
+<attribute name="REVIEWER_FURTHER" value="Joshua Kirshenbaum"/>
+<attribute name="REVIEWER_SCHEMATIC" value="Zekun Li"/>
+</part>
+<part name="U1" library="HyTechDevices" deviceset="VOLTAGE_REGULATOR_?_*" device="SOT223" technology="5V"/>
 <part name="GND7" library="HyTechSupplies" deviceset="GND" device=""/>
 <part name="P+3" library="HyTechSupplies" deviceset="+5V" device=""/>
-<part name="C11" library="HyTechDevices" deviceset="CAPACITOR_?_*" device="0603" technology="25V_0.22UF"/>
-<part name="C2" library="HyTechDevices" deviceset="CAPACITOR_?_*" device="0603" technology="10V_0.1UF"/>
+<part name="C11" library="HyTechDevices" deviceset="CAPACITOR_?_*" device="0603" technology="25V_1UF" value="CAPACITOR_0603_25V_1UF"/>
+<part name="C2" library="HyTechDevices" deviceset="CAPACITOR_?_*" device="0603" technology="10V_4.7UF" value="CAPACITOR_0603_10V_4.7UF"/>
 <part name="P+4" library="HyTechSupplies" deviceset="+12V" device=""/>
 <part name="A1" library="HyTechDevices" deviceset="TEENSY_4.0" device=""/>
@@
 <attribute name="DESCRIPTION_2" x="176.53" y="10.16" size="2.54" layer="95"/>
 </instance>
-<instance part="U1" gate="G$1" x="38.1" y="172.72" smashed="yes">
-<attribute name="NAME" x="40.64" y="165.1" size="1.778" layer="95"/>
+<instance part="U1" gate="G$1" x="30.48" y="175.26" smashed="yes">
+<attribute name="NAME" x="33.02" y="167.64" size="1.778" layer="95"/>
 </instance>
 <instance part="GND7" gate="1" x="38.1" y="160.02" smashed="yes">
@@
 </instance>
 <instance part="P+3" gate="1" x="50.8" y="177.8" smashed="yes">
-<attribute name="VALUE" x="53.34" y="180.34" size="1.778" layer="96" rot="R180"/>
+<attribute name="VALUE" x="50.8" y="180.34" size="1.778" layer="96" align="bottom-center"/>
 </instance>
 <instance part="C11" gate="G$1" x="25.4" y="170.18" smashed="yes" rot="R90">
@@
 <pinref part="GND7" gate="1" pin="GND"/>
 <pinref part="U1" gate="G$1" pin="GND"/>
-<wire x1="38.1" y1="162.56" x2="38.1" y2="165.1" width="0.1524" layer="91"/>
+<wire x1="38.1" y1="162.56" x2="50.8" y2="162.56" width="0.1524" layer="91"/>
+<junction x="38.1" y="162.56"/>
 <pinref part="C2" gate="G$1" pin="2"/>
-<wire x1="50.8" y1="165.1" x2="38.1" y2="165.1" width="0.1524" layer="91"/>
-<junction x="38.1" y="165.1"/>
+<wire x1="50.8" y1="162.56" x2="50.8" y2="165.1" width="0.1524" layer="91"/>
 <pinref part="C11" gate="G$1" pin="2"/>
-<wire x1="38.1" y1="165.1" x2="25.4" y2="165.1" width="0.1524" layer="91"/>
+<wire x1="25.4" y1="165.1" x2="25.4" y2="162.56" width="0.1524" layer="91"/>
+<wire x1="25.4" y1="162.56" x2="38.1" y2="162.56" width="0.1524" layer="91"/>
 </segment>
 <segment>
@@
 <wire x1="50.8" y1="175.26" x2="50.8" y2="172.72" width="0.1524" layer="91"/>
 <pinref part="U1" gate="G$1" pin="OUT"/>
-<wire x1="45.72" y1="172.72" x2="50.8" y2="172.72" width="0.1524" layer="91"/>
+<wire x1="48.26" y1="172.72" x2="50.8" y2="172.72" width="0.1524" layer="91"/>
 <junction x="50.8" y="172.72"/>
 </segment>
@@
 <segment>
 <pinref part="U1" gate="G$1" pin="IN"/>
-<wire x1="30.48" y1="172.72" x2="25.4" y2="172.72" width="0.1524" layer="91"/>
+<wire x1="27.94" y1="172.72" x2="25.4" y2="172.72" width="0.1524" layer="91"/>
 <wire x1="25.4" y1="172.72" x2="25.4" y2="175.26" width="0.1524" layer="91"/>
 <pinref part="C11" gate="G$1" pin="1"/>
