File: EAGLE Board Designs/Accumulator Control Unit/ACU rev1.sch (EAGLE design)
At the start: 174 parts, among them J1 CONNECTOR-CAN_MF_T_V_, J2 CONNECTOR-8_MF_T_V_, J3 CONNECTOR-8_MF_T_V_, J4 CONNECTOR-2_MF_T_V_, J5 CONNECTOR-12_MF_T_V_, Q1 TRANSISTOR_N_MOS__PMV15ENEA, Q2 TRANSISTOR_N_MOS__PMV15ENEA, T1 TRANSFORMER_HM2112ZNLT_AIRGAP, U1 VOLTAGE_REGULATOR_SOT89_12V, U10 OPAMP_1_CHANNEL_OPA991, U11 LOGICGATE_AND_DCK3, U12 OPAMP_1_CHANNEL_OPA991, U13 OPAMP_1_CHANNEL_OPA991, U14 OPAMP_1_CHANNEL_OPA991, U15 LOGICGATE_AND_DCK3, U18 OPAMP_1_CHANNEL_OPA991, U19 MAX7404, U2 ADG1423, U20 OPAMP_1_CHANNEL_OPA991, U22 OPAMP_1_CHANNEL_OPA991, U25 TCAN1051HQV-Q1, U26 MAX7404, U27 OPAMP_1_CHANNEL_OPA991, U28 MAX7404, U29 OPAMP_1_CHANNEL_OPA991, U3 LM555, U30 MAX7404, U4 OPAMP_1_CHANNEL_OPA991, U5 LTC6820, U6 ADM823, U7 OPAMP_1_CHANNEL_OPA991, U8 LOGICGATE_AND_DCK3, U9 OPAMP_1_CHANNEL_OPA991

Commit message: some placements
Parts:
- removed U1: VOLTAGE_REGULATOR_SOT89_12V, HyTechDevices:VOLTAGE_REGULATOR_SOT89_12V
- added A2: VOLTAGE_REGULATOR_MODULE_OKI-78SR_5V, HyTechDevices - Copy:VOLTAGE_REGULATOR_MODULE_OKI-78SR_5V
- added A3: VOLTAGE_REGULATOR_MODULE_OKI-78SR_3.3V, HyTechDevices - Copy:VOLTAGE_REGULATOR_MODULE_OKI-78SR_3.3V
- added C10, C9: CAPACITOR_0603_25V_10UF, HyTechDevices:CAPACITOR_0603_25V_10UF
Connections:
- net +12V: now also A2.IN, A3.IN, C9.1; no longer U1.IN
- net +3V3: now also A3.OUT, C10.1
- net +5V: now also A2.OUT; no longer U1.OUT
- net GND: now also A2.GND, A3.GND, C10.2, C9.2; no longer U1.GND
Changed lines of the file:
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@@
 <drawing>
 <settings>
-<setting alwaysvectorfont="no"/>
+<setting alwaysvectorfont="yes"/>
 <setting verticaltext="up"/>
 </settings>
@@
 <part name="P6" library="HyTechSupplies" deviceset="+12V" device=""/>
 <part name="P11" library="HyTechSupplies" deviceset="GND" device=""/>
-<part name="U1" library="HyTechDevices" deviceset="VOLTAGE_REGULATOR_?_*" device="SOT89" technology="12V"/>
 <part name="C1" library="HyTechDevices" deviceset="CAPACITOR_?_*" device="0603" technology="25V_10UF"/>
 <part name="C2" library="HyTechDevices" deviceset="CAPACITOR_?_*" device="0603" technology="25V_10UF"/>
@@
 <part name="P4" library="HyTechSupplies" deviceset="GND" device=""/>
 <part name="J2" library="HyTechDevices - Copy" deviceset="CONNECTOR-8_?_*" device="MF_T_V"/>
+<part name="A2" library="HyTechDevices - Copy" deviceset="VOLTAGE_REGULATOR_MODULE_?_*" device="OKI-78SR" technology="5V"/>
+<part name="C9" library="HyTechDevices" deviceset="CAPACITOR_?_*" device="0603" technology="25V_10UF"/>
+<part name="C10" library="HyTechDevices" deviceset="CAPACITOR_?_*" device="0603" technology="25V_10UF"/>
+<part name="P41" library="HyTechSupplies" deviceset="GND" device=""/>
+<part name="P42" library="HyTechSupplies" deviceset="+12V" device=""/>
+<part name="P43" library="HyTechSupplies" deviceset="+3V3" device=""/>
+<part name="A3" library="HyTechDevices - Copy" deviceset="VOLTAGE_REGULATOR_MODULE_?_*" device="OKI-78SR" technology="3.3V"/>
 </parts>
 <sheets>
@@
 <attribute name="VALUE" x="88.9" y="176.53" size="1.27" layer="96" align="top-center"/>
 </instance>
-<instance part="U1" gate="G$1" x="154.94" y="195.58" smashed="yes">
-<attribute name="NAME" x="154.94" y="196.342" size="1.27" layer="95"/>
-<attribute name="MPN" x="163.83" y="184.658" size="1.27" layer="96" align="top-left"/>
-</instance>
 <instance part="C1" gate="G$1" x="147.32" y="187.96" smashed="yes" rot="R90">
 <attribute name="NAME" x="144.78" y="186.69" size="1.27" layer="95" rot="R90" align="bottom-center"/>
@@
 <attribute name="NAME" x="58.42" y="135.382" size="1.27" layer="95"/>
 <attribute name="MPN" x="58.42" y="111.125" size="1.27" layer="96" align="top-left"/>
+</instance>
+<instance part="A2" gate="G$1" x="154.94" y="195.58" smashed="yes">
+<attribute name="NAME" x="154.94" y="196.342" size="1.27" layer="95"/>
+<attribute name="MPN" x="163.83" y="184.658" size="1.27" layer="96" align="top-left"/>
+</instance>
+<instance part="C9" gate="G$1" x="147.32" y="157.48" smashed="yes" rot="R90">
+<attribute name="NAME" x="144.78" y="156.21" size="1.27" layer="95" rot="R90" align="bottom-center"/>
+<attribute name="VOLTAGE" x="149.86" y="156.21" size="1.27" layer="96" rot="R90" align="top-center"/>
+<attribute name="CAPACITANCE" x="151.638" y="156.21" size="1.27" layer="96" rot="R90" align="top-center"/>
+</instance>
+<instance part="C10" gate="G$1" x="177.8" y="157.48" smashed="yes" rot="R90">
+<attribute name="NAME" x="175.26" y="156.21" size="1.27" layer="95" rot="R90" align="bottom-center"/>
+<attribute name="VOLTAGE" x="180.34" y="156.21" size="1.27" layer="96" rot="R90" align="top-center"/>
+<attribute name="CAPACITANCE" x="182.118" y="156.21" size="1.27" layer="96" rot="R90" align="top-center"/>
+</instance>
+<instance part="P41" gate="1" x="162.56" y="144.78" smashed="yes">
+<attribute name="VALUE" x="162.56" y="143.51" size="1.27" layer="96" align="top-center"/>
+</instance>
+<instance part="P42" gate="1" x="144.78" y="167.64" smashed="yes">
+<attribute name="VALUE" x="144.78" y="171.45" size="1.27" layer="96" align="bottom-center"/>
+</instance>
+<instance part="P43" gate="G$1" x="180.34" y="167.64" smashed="yes">
+<attribute name="VALUE" x="180.34" y="168.91" size="1.27" layer="96" align="bottom-center"/>
+</instance>
+<instance part="A3" gate="G$1" x="154.94" y="165.1" smashed="yes">
+<attribute name="NAME" x="154.94" y="165.862" size="1.27" layer="95"/>
+<attribute name="MPN" x="163.83" y="154.178" size="1.27" layer="96" align="top-left"/>
 </instance>
 </instances>
@@
 <net name="+5V" class="0">
 <segment>
-<pinref part="U1" gate="G$1" pin="OUT"/>
 <wire x1="172.72" y1="193.04" x2="177.8" y2="193.04" width="0.1524" layer="91"/>
 <wire x1="177.8" y1="193.04" x2="180.34" y2="193.04" width="0.1524" layer="91"/>
@@
 <junction x="177.8" y="193.04"/>
 <pinref part="P14" gate="1" pin="+5V"/>
+<pinref part="A2" gate="G$1" pin="OUT"/>
 </segment>
 <segment>
@@
 </segment>
 <segment>
-<pinref part="U1" gate="G$1" pin="GND"/>
 <wire x1="162.56" y1="182.88" x2="162.56" y2="180.34" width="0.1524" layer="91"/>
 <wire x1="162.56" y1="177.8" x2="162.56" y2="180.34" width="0.1524" layer="91"/>
@@
 <wire x1="177.8" y1="180.34" x2="177.8" y2="182.88" width="0.1524" layer="91"/>
 <pinref part="P12" gate="1" pin="GND"/>
+<pinref part="A2" gate="G$1" pin="GND"/>
 </segment>
 <segment>
@@
 <wire x1="38.1" y1="104.14" x2="38.1" y2="101.6" width="0.1524" layer="91"/>
 </segment>
+<segment>
+<wire x1="162.56" y1="152.4" x2="162.56" y2="149.86" width="0.1524" layer="91"/>
+<wire x1="162.56" y1="147.32" x2="162.56" y2="149.86" width="0.1524" layer="91"/>
+<junction x="162.56" y="149.86"/>
+<wire x1="162.56" y1="149.86" x2="177.8" y2="149.86" width="0.1524" layer="91"/>
+<pinref part="C9" gate="G$1" pin="2"/>
+<wire x1="147.32" y1="152.4" x2="147.32" y2="149.86" width="0.1524" layer="91"/>
+<wire x1="147.32" y1="149.86" x2="162.56" y2="149.86" width="0.1524" layer="91"/>
+<pinref part="C10" gate="G$1" pin="2"/>
+<wire x1="177.8" y1="149.86" x2="177.8" y2="152.4" width="0.1524" layer="91"/>
+<pinref part="P41" gate="1" pin="GND"/>
+<pinref part="A3" gate="G$1" pin="GND"/>
+</segment>
 </net>
 <net name="+12V" class="0">
@@
 </segment>
 <segment>
-<pinref part="U1" gate="G$1" pin="IN"/>
 <wire x1="152.4" y1="193.04" x2="147.32" y2="193.04" width="0.1524" layer="91"/>
 <wire x1="147.32" y1="193.04" x2="144.78" y2="193.04" width="0.1524" layer="91"/>
@@
 <junction x="147.32" y="193.04"/>
 <pinref part="P13" gate="1" pin="+12V"/>
+<pinref part="A2" gate="G$1" pin="IN"/>
 </segment>
 <segment>
@@
 <pinref part="U$1" gate="G$1" pin="1"/>
 </segment>
+<segment>
+<wire x1="152.4" y1="162.56" x2="147.32" y2="162.56" width="0.1524" layer="91"/>
+<wire x1="147.32" y1="162.56" x2="144.78" y2="162.56" width="0.1524" layer="91"/>
+<wire x1="144.78" y1="162.56" x2="144.78" y2="165.1" width="0.1524" layer="91"/>
+<pinref part="C9" gate="G$1" pin="1"/>
+<wire x1="147.32" y1="160.02" x2="147.32" y2="162.56" width="0.1524" layer="91"/>
+<junction x="147.32" y="162.56"/>
+<pinref part="P42" gate="1" pin="+12V"/>
+<pinref part="A3" gate="G$1" pin="IN"/>
+</segment>
 </net>
 <net name="BSPD_CURRENT" class="0">
@@
 <wire x1="210.82" y1="182.88" x2="210.82" y2="190.5" width="0.1524" layer="91"/>
 </segment>
-</net>
+<segment>
+<wire x1="172.72" y1="162.56" x2="177.8" y2="162.56" width="0.1524" layer="91"/>
+<wire x1="177.8" y1="162.56" x2="180.34" y2="162.56" width="0.1524" layer="91"/>
+<wire x1="180.34" y1="162.56" x2="180.34" y2="165.1" width="0.1524" layer="91"/>
+<pinref part="C10" gate="G$1" pin="1"/>
+<wire x1="177.8" y1="160.02" x2="177.8" y2="162.56" width="0.1524" layer="91"/>
+<junction x="177.8" y="162.56"/>
+<pinref part="P43" gate="G$1" pin="+3V3"/>
+<pinref part="A3" gate="G$1" pin="OUT"/>
+</segment>
+</net>

Commit message: more placements and routing
Connections:
- net +12V: now also U$1.7; no longer U$1.1
- net ACCUMULATOR_GND: now also U$1.14; no longer U$1.9
- net BSPD_CURRENT_TEENSY: now also A1.A8; no longer A1.A6
- net CANH: now also J5.9, U$1.3; no longer J5.8, U$1.2
- net CANL: now also J5.8, U$1.2; no longer J5.9, U$1.3
- net CURRENT: now also U$1.8; no longer U$1.6
- net CURRENT_FILTERED: now also A1.A7; no longer A1.A0
- net CURRENT_REF: now also U$1.9; no longer U$1.7
- net CURRENT_REF_FILTERED: now also A1.A6; no longer A1.A1
- net GND: now also U$1.6; no longer U$1.8
- net MHS_TEENSY: now also A1.A1; no longer A1.A8
- net PRECHARGE_OK_TEENSY: now also A1.A0; no longer A1.A7
Changed lines of the file:
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@@
 <part name="P7" library="HyTechSupplies" deviceset="+5V" device=""/>
 <part name="P8" library="HyTechSupplies" deviceset="+12V" device=""/>
-<part name="P9" library="HyTechSupplies" deviceset="GND" device=""/>
 <part name="P86" library="HyTechSupplies" deviceset="GND" device=""/>
 <part name="R46" library="HyTechDevices - Copy" deviceset="RESISTOR_?_*" device="0603" technology="2.2K"/>
-<part name="P3" library="HyTechSupplies" deviceset="+12V" device=""/>
 <part name="P4" library="HyTechSupplies" deviceset="GND" device=""/>
 <part name="J2" library="HyTechDevices - Copy" deviceset="CONNECTOR-8_?_*" device="MF_T_V"/>
@@
 <part name="P43" library="HyTechSupplies" deviceset="+3V3" device=""/>
 <part name="A3" library="HyTechDevices - Copy" deviceset="VOLTAGE_REGULATOR_MODULE_?_*" device="OKI-78SR" technology="3.3V"/>
+<part name="P9" library="HyTechSupplies" deviceset="GND" device=""/>
+<part name="P3" library="HyTechSupplies" deviceset="+12V" device=""/>
 </parts>
 <sheets>
@@
 <attribute name="MPN" x="10.16" y="93.345" size="1.27" layer="96" align="top-left"/>
 </instance>
-<instance part="P7" gate="1" x="38.1" y="127" smashed="yes">
-<attribute name="VALUE" x="38.1" y="129.54" size="1.27" layer="96" align="bottom-center"/>
-</instance>
+<instance part="P7" gate="1" x="38.1" y="127" smashed="yes"/>
 <instance part="P8" gate="1" x="78.74" y="137.16" smashed="yes">
 <attribute name="VALUE" x="78.74" y="140.97" size="1.27" layer="96" align="bottom-center"/>
 </instance>
-<instance part="P9" gate="1" x="48.26" y="109.22" smashed="yes">
-<attribute name="VALUE" x="48.26" y="107.95" size="1.27" layer="96" align="top-center"/>
-</instance>
 <instance part="P86" gate="1" x="93.98" y="111.76" smashed="yes">
 <attribute name="VALUE" x="93.98" y="110.49" size="1.27" layer="96" align="top-center"/>
@@
 <attribute name="RESISTANCE" x="95.25" y="120.65" size="1.27" layer="96" rot="R90" align="top-center"/>
 </instance>
-<instance part="P3" gate="1" x="48.26" y="132.08" smashed="yes">
-<attribute name="VALUE" x="48.26" y="135.89" size="1.27" layer="96" align="bottom-center"/>
-</instance>
 <instance part="P4" gate="1" x="43.18" y="119.38" smashed="yes">
 <attribute name="VALUE" x="43.18" y="118.11" size="1.27" layer="96" align="top-center"/>
@@
 <attribute name="MPN" x="163.83" y="154.178" size="1.27" layer="96" align="top-left"/>
 </instance>
+<instance part="P9" gate="1" x="48.26" y="114.3" smashed="yes">
+<attribute name="VALUE" x="48.26" y="113.03" size="1.27" layer="96" align="top-center"/>
+</instance>
+<instance part="P3" gate="1" x="53.34" y="116.84" smashed="yes">
+<attribute name="VALUE" x="53.34" y="120.65" size="1.27" layer="96" align="bottom-center"/>
+</instance>
 </instances>
 <busses>
@@
 </segment>
 <segment>
-<wire x1="68.58" y1="167.64" x2="71.12" y2="167.64" width="0.1524" layer="91"/>
-<label x="71.12" y="167.64" size="1.27" layer="95" xref="yes"/>
-<pinref part="J5" gate="G$1" pin="8"/>
+<wire x1="68.58" y1="165.1" x2="71.12" y2="165.1" width="0.1524" layer="91"/>
+<label x="71.12" y="165.1" size="1.27" layer="95" xref="yes"/>
+<pinref part="J5" gate="G$1" pin="9"/>
 </segment>
 <segment>
-<wire x1="20.32" y1="127" x2="22.86" y2="127" width="0.1524" layer="91"/>
-<label x="22.86" y="127" size="1.27" layer="95" xref="yes"/>
-<pinref part="U$1" gate="G$1" pin="2"/>
+<wire x1="20.32" y1="124.46" x2="22.86" y2="124.46" width="0.1524" layer="91"/>
+<label x="22.86" y="124.46" size="1.27" layer="95" xref="yes"/>
+<pinref part="U$1" gate="G$1" pin="3"/>
 </segment>
 </net>
@@
 </segment>
 <segment>
-<wire x1="68.58" y1="165.1" x2="71.12" y2="165.1" width="0.1524" layer="91"/>
-<label x="71.12" y="165.1" size="1.27" layer="95" xref="yes"/>
-<pinref part="J5" gate="G$1" pin="9"/>
+<wire x1="68.58" y1="167.64" x2="71.12" y2="167.64" width="0.1524" layer="91"/>
+<label x="71.12" y="167.64" size="1.27" layer="95" xref="yes"/>
+<pinref part="J5" gate="G$1" pin="8"/>
 </segment>
 <segment>
-<wire x1="20.32" y1="124.46" x2="22.86" y2="124.46" width="0.1524" layer="91"/>
-<label x="22.86" y="124.46" size="1.27" layer="95" xref="yes"/>
-<pinref part="U$1" gate="G$1" pin="3"/>
+<wire x1="20.32" y1="127" x2="22.86" y2="127" width="0.1524" layer="91"/>
+<label x="22.86" y="127" size="1.27" layer="95" xref="yes"/>
+<pinref part="U$1" gate="G$1" pin="2"/>
 </segment>
 </net>
@@
 </segment>
 <segment>
-<wire x1="20.32" y1="111.76" x2="48.26" y2="111.76" width="0.1524" layer="91"/>
-<pinref part="P9" gate="1" pin="GND"/>
-<pinref part="U$1" gate="G$1" pin="8"/>
-</segment>
-<segment>
 <pinref part="R46" gate="G$1" pin="1"/>
 <pinref part="P86" gate="1" pin="GND"/>
@@
 <pinref part="A3" gate="G$1" pin="GND"/>
 </segment>
+<segment>
+<wire x1="20.32" y1="116.84" x2="48.26" y2="116.84" width="0.1524" layer="91"/>
+<pinref part="P9" gate="1" pin="GND"/>
+<pinref part="U$1" gate="G$1" pin="6"/>
+</segment>
 </net>
 <net name="+12V" class="0">
@@
 </segment>
 <segment>
-<wire x1="20.32" y1="129.54" x2="48.26" y2="129.54" width="0.1524" layer="91"/>
-<pinref part="P3" gate="1" pin="+12V"/>
-<pinref part="U$1" gate="G$1" pin="1"/>
-</segment>
-<segment>
 <wire x1="152.4" y1="162.56" x2="147.32" y2="162.56" width="0.1524" layer="91"/>
 <wire x1="147.32" y1="162.56" x2="144.78" y2="162.56" width="0.1524" layer="91"/>
@@
 <pinref part="A3" gate="G$1" pin="IN"/>
 </segment>
+<segment>
+<wire x1="20.32" y1="114.3" x2="53.34" y2="114.3" width="0.1524" layer="91"/>
+<pinref part="P3" gate="1" pin="+12V"/>
+<pinref part="U$1" gate="G$1" pin="7"/>
+</segment>
 </net>
 <net name="BSPD_CURRENT" class="0">
@@
 </segment>
 <segment>
-<pinref part="U$1" gate="G$1" pin="9"/>
-<wire x1="20.32" y1="109.22" x2="22.86" y2="109.22" width="0.1524" layer="91"/>
-<label x="22.86" y="109.22" size="1.27" layer="95" xref="yes"/>
+<wire x1="20.32" y1="96.52" x2="22.86" y2="96.52" width="0.1524" layer="91"/>
+<label x="22.86" y="96.52" size="1.27" layer="95" xref="yes"/>
+<pinref part="U$1" gate="G$1" pin="14"/>
 </segment>
 </net>
@@
 </segment>
 </net>
-<net name="CURRENT_REF" class="0">
-<segment>
-<wire x1="20.32" y1="114.3" x2="22.86" y2="114.3" width="0.1524" layer="91"/>
-<label x="22.86" y="114.3" size="1.27" layer="95" xref="yes"/>
-<pinref part="U$1" gate="G$1" pin="7"/>
-</segment>
-</net>
-<net name="CURRENT" class="0">
-<segment>
-<wire x1="20.32" y1="116.84" x2="22.86" y2="116.84" width="0.1524" layer="91"/>
-<label x="22.86" y="116.84" size="1.27" layer="95" xref="yes"/>
-<pinref part="U$1" gate="G$1" pin="6"/>
-</segment>
-</net>
 <net name="MHS" class="0">
 <segment>
@@
 </segment>
 </net>
+<net name="CURRENT_REF" class="0">
+<segment>
+<wire x1="20.32" y1="109.22" x2="22.86" y2="109.22" width="0.1524" layer="91"/>
+<label x="22.86" y="109.22" size="1.27" layer="95" xref="yes"/>
+<pinref part="U$1" gate="G$1" pin="9"/>
+</segment>
+</net>
+<net name="CURRENT" class="0">
+<segment>
+<wire x1="20.32" y1="111.76" x2="22.86" y2="111.76" width="0.1524" layer="91"/>
+<label x="22.86" y="111.76" size="1.27" layer="95" xref="yes"/>
+<pinref part="U$1" gate="G$1" pin="8"/>
+</segment>
+</net>
 </nets>
 </sheet>
@@
 </segment>
 <segment>
-<pinref part="A1" gate="G$1" pin="A7"/>
-<wire x1="48.26" y1="152.4" x2="45.72" y2="152.4" width="0.1524" layer="91"/>
-<label x="45.72" y="152.4" size="1.27" layer="95" rot="R180" xref="yes"/>
+<wire x1="48.26" y1="170.18" x2="45.72" y2="170.18" width="0.1524" layer="91"/>
+<label x="45.72" y="170.18" size="1.27" layer="95" rot="R180" xref="yes"/>
+<pinref part="A1" gate="G$1" pin="A0"/>
 </segment>
 </net>
@@
 </segment>
 </net>
-<net name="CURRENT_FILTERED" class="0">
-<segment>
-<pinref part="A1" gate="G$1" pin="A0"/>
-<wire x1="48.26" y1="170.18" x2="45.72" y2="170.18" width="0.1524" layer="91"/>
-<label x="45.72" y="170.18" size="1.27" layer="95" rot="R180" xref="yes"/>
-</segment>
-</net>
-<net name="CURRENT_REF_FILTERED" class="0">
-<segment>
-<pinref part="A1" gate="G$1" pin="A1"/>
-<wire x1="48.26" y1="167.64" x2="45.72" y2="167.64" width="0.1524" layer="91"/>
-<label x="45.72" y="167.64" size="1.27" layer="95" rot="R180" xref="yes"/>
-</segment>
-</net>
 <net name="BSPD_CURRENT" class="0">
 <segment>
@@
 </segment>
 <segment>
-<pinref part="A1" gate="G$1" pin="A6"/>
-<wire x1="48.26" y1="154.94" x2="45.72" y2="154.94" width="0.1524" layer="91"/>
-<label x="45.72" y="154.94" size="1.27" layer="95" rot="R180" xref="yes"/>
+<wire x1="48.26" y1="149.86" x2="45.72" y2="149.86" width="0.1524" layer="91"/>
+<label x="45.72" y="149.86" size="1.27" layer="95" rot="R180" xref="yes"/>
+<pinref part="A1" gate="G$1" pin="A8"/>
 </segment>
 </net>
@@
 <segment>
 <pinref part="A1" gate="G$1" pin="A2"/>
-<wire x1="48.26" y1="165.1" x2="45.72" y2="165.1" width="0.1524" layer="91"/>
-<label x="45.72" y="165.1" size="1.27" layer="95" rot="R180" xref="yes"/>
+<wire x1="48.26" y1="165.1" x2="43.18" y2="165.1" width="0.1524" layer="91"/>
+<label x="43.18" y="165.1" size="1.27" layer="95" rot="R180" xref="yes"/>
 </segment>
 </net>
@@
 </segment>
 <segment>
-<pinref part="A1" gate="G$1" pin="A8"/>
-<wire x1="48.26" y1="149.86" x2="45.72" y2="149.86" width="0.1524" layer="91"/>
-<label x="45.72" y="149.86" size="1.27" layer="95" rot="R180" xref="yes"/>
+<wire x1="48.26" y1="167.64" x2="45.72" y2="167.64" width="0.1524" layer="91"/>
+<label x="45.72" y="167.64" size="1.27" layer="95" rot="R180" xref="yes"/>
+<pinref part="A1" gate="G$1" pin="A1"/>
 </segment>
 </net>
@@
 </segment>
 </net>
+<net name="CURRENT_FILTERED" class="0">
+<segment>
+<wire x1="48.26" y1="152.4" x2="45.72" y2="152.4" width="0.1524" layer="91"/>
+<label x="45.72" y="152.4" size="1.27" layer="95" rot="R180" xref="yes"/>
+<pinref part="A1" gate="G$1" pin="A7"/>
+</segment>
+</net>
+<net name="CURRENT_REF_FILTERED" class="0">
+<segment>
+<wire x1="48.26" y1="154.94" x2="45.72" y2="154.94" width="0.1524" layer="91"/>
+<label x="45.72" y="154.94" size="1.27" layer="95" rot="R180" xref="yes"/>
+<pinref part="A1" gate="G$1" pin="A6"/>
+</segment>
+</net>
