File: EAGLE Board Designs/Accumulator Control Unit/Accumulator Control Unit rev3.brd (EAGLE design)
At the start: 186.7 x 135.7 mm, 241 parts, among them J1 CONNECTOR-2_MF_T_V_, J100 CONNECTOR-8_S_S, J2 CONNECTOR-8_MF_T_V_, J3 CONNECTOR-14_MF_T_V_, J4 JUMPER__1X02, J5 CONNECTOR-12_MF_T_V_, J6 CONNECTOR-CAN_μF_S_RA_, Q1 TRANSISTOR_N_MOS__PMV15ENEA, Q100 TRANSISTOR_N_MOS__PMV15ENEA, Q101 TRANSISTOR_N_MOS__PMV15ENEA, Q2 TRANSISTOR_N_MOS__PMV15ENEA, T1 TRANSFORMER_HM2112ZNLT_AIRGAP, U1 RELAY_SOLIDSTATE_NO, U10 MAX7404, U100 ADG1423, U101 LM555, U11 OPAMP_1_CHANNEL_OPA991, U12 LOGICGATE_AND_DCK3, U13 OPAMP_1_CHANNEL_OPA991, U14 LOGICGATE_AND_DCK3, U15 OPAMP_1_CHANNEL_OPA991, U16 LOGICGATE_AND_DCK3, U17 OPAMP_1_CHANNEL_OPA991, U18 OPAMP_1_CHANNEL_OPA991, U19 MAX7404, U2 RELAY_SOLIDSTATE_NO, U20 OPAMP_1_CHANNEL_OPA991, U21 OPAMP_1_CHANNEL_OPA991, U22 OPAMP_1_CHANNEL_OPA991, U23 OPAMP_1_CHANNEL_OPA991, U24 OPAMP_1_CHANNEL_OPA991, U25 MAX7404, U26 VOLTAGE_REGULATOR_SOT223_3.3V, U27 TCAN1051HQV-Q1, U3 OPAMP_1_CHANNEL_OPA991, U4 MAX7404, U5 LTC6820, U6 LOGICGATE_BUFFER, U7 ADM8316WBX30, U8 RELAY_SOLIDSTATE_NO, U9 OPAMP_1_CHANNEL_OPA991

Commit message: some changes
Parts:
- R106: value RESISTOR_0603_1K -> RESISTOR_0603_10K
- WATCHDOG: value LED_0603_GREEN -> LED_0603_BLUE
Changed lines of the file:
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@@
 <attribute name="VOLTAGE_MAX" value="75V" x="149.86590625" y="105.78148125" size="1.778" layer="27" rot="R90" display="off"/>
 </element>
-<element name="R106" library="HyTechDevices" package="0603-RES" value="RESISTOR_0603_1K" x="5.78529375" y="21.72651875" smashed="yes" rot="MR0">
-<attribute name="DKPN" value="311-1.00KHRCT-ND" x="-55.17470625" y="-65.90348125" size="1.778" layer="28" rot="MR0" display="off"/>
+<element name="R106" library="HyTechDevices" package="0603-RES" value="RESISTOR_0603_10K" x="5.78529375" y="21.72651875" smashed="yes" rot="MR0">
+<attribute name="DKPN" value="311-10.0KHRCT-ND" x="-55.17470625" y="-65.90348125" size="1.778" layer="28" rot="MR0" display="off"/>
 <attribute name="MANUFACTURER" value="Yageo" x="-55.17470625" y="-65.90348125" size="1.778" layer="28" rot="MR0" display="off"/>
-<attribute name="MOPN" value="603-RC0603FR-071KL" x="-55.17470625" y="-65.90348125" size="1.778" layer="28" rot="MR0" display="off"/>
-<attribute name="MPN" value="RC0603FR-071KL" x="-55.17470625" y="-65.90348125" size="1.778" layer="28" rot="MR0" display="off"/>
+<attribute name="MOPN" value="603-RC0603FR-0710KL" x="-55.17470625" y="-65.90348125" size="1.778" layer="28" rot="MR0" display="off"/>
+<attribute name="MPN" value="RC0603FR-0710KL" x="-55.17470625" y="-65.90348125" size="1.778" layer="28" rot="MR0" display="off"/>
 <attribute name="NAME" x="5.78529375" y="22.36151875" size="0.8128" layer="26" font="vector" rot="MR0" align="bottom-center"/>
 <attribute name="POWER" value="0.1W" x="-55.17470625" y="-65.90348125" size="1.778" layer="28" rot="MR0" display="off"/>
-<attribute name="RESISTANCE" value="1k" x="-55.17470625" y="-65.90348125" size="1.778" layer="28" rot="MR0" display="off"/>
+<attribute name="RESISTANCE" value="10k" x="-55.17470625" y="-65.90348125" size="1.778" layer="28" rot="MR0" display="off"/>
 <attribute name="TOLERANCE" value="1%" x="-55.17470625" y="-65.90348125" size="1.778" layer="28" rot="MR0" display="off"/>
-<attribute name="VOLTAGE_CONTINUOUS" value="10.00V" x="-55.17470625" y="-65.90348125" size="1.778" layer="28" rot="MR0" display="off"/>
+<attribute name="VOLTAGE_CONTINUOUS" value="31.62V" x="-55.17470625" y="-65.90348125" size="1.778" layer="28" rot="MR0" display="off"/>
 <attribute name="VOLTAGE_MAX" value="75V" x="-55.17470625" y="-65.90348125" size="1.778" layer="28" rot="MR0" display="off"/>
 </element>
@@
 <attribute name="VOLTAGE_MAX" value="75V" x="18.288" y="23.622" size="1.778" layer="27" rot="R270" display="off"/>
 </element>
-<element name="WATCHDOG" library="HyTechDevices" package="0603-LED" value="LED_0603_GREEN" x="167.386" y="67.7926" smashed="yes" rot="R270">
-<attribute name="COLOR" value="Green" x="167.386" y="67.7926" size="1.778" layer="27" rot="R270" display="off"/>
-<attribute name="DKPN" value="754-1790-1-ND" x="167.386" y="67.7926" size="1.778" layer="27" rot="R270" display="off"/>
+<element name="WATCHDOG" library="HyTechDevices" package="0603-LED" value="LED_0603_BLUE" x="167.386" y="67.7926" smashed="yes" rot="R270">
+<attribute name="COLOR" value="Blue" x="167.386" y="67.7926" size="1.778" layer="27" rot="R270" display="off"/>
+<attribute name="DKPN" value="754-1789-1-ND" x="167.386" y="67.7926" size="1.778" layer="27" rot="R270" display="off"/>
 <attribute name="MANUFACTURER" value="Kingbright" x="167.386" y="67.7926" size="1.778" layer="27" rot="R270" display="off"/>
-<attribute name="MOPN" value="604-APT1608ZGCK" x="167.386" y="67.7926" size="1.778" layer="27" rot="R270" display="off"/>
-<attribute name="MPN" value="APT1608ZGCK" x="167.386" y="67.7926" size="1.778" layer="27" rot="R270" display="off"/>
+<attribute name="MOPN" value="604-APT1608VBC/D" x="167.386" y="67.7926" size="1.778" layer="27" rot="R270" display="off"/>
+<attribute name="MPN" value="APT1608VBC/D" x="167.386" y="67.7926" size="1.778" layer="27" rot="R270" display="off"/>
 <attribute name="NAME" x="166.509" y="67.7418" size="0.8128" layer="25" font="vector" rot="R90" align="bottom-center"/>
 </element>
@@
 <contactref element="U7" pad="3"/>
 <contactref element="R27" pad="2"/>
-<wire x1="161.76509375" y1="62.36309375" x2="161.798" y2="62.396" width="0.1524" layer="1"/>
 <wire x1="161.798" y1="62.396" x2="163.6647875" y2="62.396" width="0.1524" layer="1"/>
 <wire x1="163.6647875" y1="62.396" x2="163.80030625" y2="62.26048125" width="0.1524" layer="1"/>
