File: EAGLE Board Designs/Tractive System Board/Tractive System Board Rev1.brd (EAGLE design)
At the start: 206.7 x 150.3 mm, 193 parts, among them J3 CONNECTOR-8_MF_T_V_, J5 CONNECTOR-4__, K4 RELAY_SPST_NC_POLARIZED_3550_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, K5 RELAY_SPST_NO_3550_12, Q2 TRANSISTOR_N_MOS__PMV15ENEA, U1 LTC6994_1, U10 DCM4623TD2J13D0T70, U11 RELAY_SOLIDSTATE_NC_AG, U15 LOGICGATE_INVERTER_DCKR, U16 LTC3639, U17 VOLTAGE_REGULATOR_ADJ_LR8_DPAK, U18 ISO224B_AIRGAP, U19 ISO224B_AIRGAP, U2 VOLTAGE_REGULATOR_SOT223_5V

Commit message: some changes
Parts:
- removed D14: LED_0603_ORANGE, HyTechDevices:0603-LED
- removed R56: RESISTOR_0603_1K, HyTechDevices:0603-RES
- added C10: CAPACITOR_0603_10V_0.1UF, HyTechDevices:0603-CAP
Connections:
- removed net N$1: D14.2, R56.1
- net +5V: now also C10.1
- net ENABLE: no longer R56.2
- net GND: now also C10.2
- net TS-FUSED: no longer D14.1, U11.3
Routing:
- net TS-FUSED: track 653.0 -> 646.7 mm
- net N$1: track 1.23 -> 0.00 mm
- net ENABLE: track 70.8 -> 70.0 mm
Changed lines of the file:
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@@
 <drawing>
 <settings>
-<setting alwaysvectorfont="yes"/>
+<setting alwaysvectorfont="no"/>
 <setting verticaltext="up"/>
 </settings>
@@
 <attribute name="VOLTAGE" value="500V" x="125.3255" y="70.62036875" size="1.778" layer="27" font="vector" rot="R180" display="off"/>
 </element>
-<element name="R56" library="HyTechDevices" package="0603-RES" value="RESISTOR_0603_1K" x="80.304003125" y="70.8718" smashed="yes" rot="R180">
-<attribute name="DKPN" value="311-1.00KHRCT-ND" x="79.66289375" y="70.8718" size="1.778" layer="27" rot="R180" display="off"/>
-<attribute name="MANUFACTURER" value="Yageo" x="79.66289375" y="70.8718" size="1.778" layer="27" rot="R180" display="off"/>
-<attribute name="MOPN" value="603-RC0603FR-071KL" x="79.66289375" y="70.8718" size="1.778" layer="27" rot="R180" display="off"/>
-<attribute name="MPN" value="RC0603FR-071KL" x="79.66289375" y="70.8718" size="1.778" layer="27" rot="R180" display="off"/>
-<attribute name="NAME" x="80.304003125" y="70.2368" size="0.8128" layer="25" font="vector" rot="R180" align="bottom-center"/>
-<attribute name="POWER" value="0.1W" x="79.66289375" y="70.8718" size="1.778" layer="27" rot="R180" display="off"/>
-<attribute name="RESISTANCE" value="1k" x="79.66289375" y="70.8718" size="1.778" layer="27" rot="R180" display="off"/>
-<attribute name="TOLERANCE" value="1%" x="79.66289375" y="70.8718" size="1.778" layer="27" rot="R180" display="off"/>
-<attribute name="VOLTAGE_CONTINUOUS" value="10.00V" x="79.66289375" y="70.8718" size="1.778" layer="27" rot="R180" display="off"/>
-<attribute name="VOLTAGE_MAX" value="75V" x="79.66289375" y="70.8718" size="1.778" layer="27" rot="R180" display="off"/>
-</element>
-<element name="D14" library="HyTechDevices" package="0603-LED" value="LED_0603_ORANGE" x="83.198003125" y="70.88723125" smashed="yes" rot="R180">
-<attribute name="COLOR" value="Orange" x="82.45689375" y="70.88723125" size="1.778" layer="27" rot="R180" display="off"/>
-<attribute name="DKPN" value="754-1120-1-ND" x="82.45689375" y="70.88723125" size="1.778" layer="27" rot="R180" display="off"/>
-<attribute name="MANUFACTURER" value="Kingbright" x="82.45689375" y="70.88723125" size="1.778" layer="27" rot="R180" display="off"/>
-<attribute name="MOPN" value="604-APT1608SECK" x="82.45689375" y="70.88723125" size="1.778" layer="27" rot="R180" display="off"/>
-<attribute name="MPN" value="APT1608SECK" x="82.45689375" y="70.88723125" size="1.778" layer="27" rot="R180" display="off"/>
-<attribute name="NAME" x="83.198003125" y="70.13723125" size="0.8128" layer="25" font="vector" rot="R180" align="bottom-center"/>
-</element>
 <element name="U$31" library="HyTechDevices" package="MOLEX_MICROFIT_PTH_VERTICAL_06_SINGLE_SPACED" value="CONNECTOR-5_6_SPACED_" x="198.671275" y="51.9166625" smashed="yes" rot="R270">
 <attribute name="NAME" x="196.385275" y="51.9166625" size="0.8128" layer="25" rot="R90" align="bottom-center"/>
@@
 <element name="U$69" library="HyTechAesthetics" package="TS" value="" x="2.54" y="10.668" smashed="yes"/>
 <element name="U$54" library="HyTechAesthetics" package="LOGO_GT_0.50&quot;" value="" x="127" y="116.84" smashed="yes"/>
+<element name="C10" library="HyTechDevices" package="0603-CAP" value="CAPACITOR_0603_10V_0.1UF" x="2.54" y="-7.62" smashed="yes">
+<attribute name="CAPACITANCE" value="0.1µF" x="2.54" y="-7.62" size="1.778" layer="27" display="off"/>
+<attribute name="DKPN" value="720-1688-1-ND" x="2.54" y="-7.62" size="1.778" layer="27" display="off"/>
+<attribute name="MANUFACTURER" value="Vishay Vitramon" x="2.54" y="-7.62" size="1.778" layer="27" display="off"/>
+<attribute name="MOPN" value="77-VJ0603Y104JXQPBC" x="2.54" y="-7.62" size="1.778" layer="27" display="off"/>
+<attribute name="MPN" value="VJ0603Y104JXQPW1BC" x="2.54" y="-7.62" size="1.778" layer="27" display="off"/>
+<attribute name="NAME" x="2.54" y="-6.87" size="0.8128" layer="25" font="vector" align="bottom-center"/>
+<attribute name="TOLERANCE" value="5%" x="2.54" y="-7.62" size="1.778" layer="27" display="off"/>
+<attribute name="VOLTAGE" value="10V" x="2.54" y="-7.62" size="1.778" layer="27" display="off"/>
+</element>
 </elements>
 <signals>
@@
 <wire x1="56.369" y1="8.978" x2="57.389" y2="7.958" width="0.254" layer="1"/>
 <wire x1="87.40103125" y1="8.87696875" x2="88.15" y2="8.128" width="0.254" layer="16"/>
+<contactref element="C10" pad="2"/>
+<wire x1="128.31" y1="15.748" x2="191.516" y2="3.851" width="0" layer="19" extent="1-16"/>
+<wire x1="126.626115625" y1="15.805925" x2="128.31" y2="15.748" width="0" layer="19" extent="16-16"/>
+<wire x1="95.516" y1="8.001" x2="126.626115625" y2="15.805925" width="0" layer="19" extent="16-16"/>
+<wire x1="88.15" y1="8.128" x2="93.218" y2="8.128" width="0" layer="19" extent="16-16"/>
+<wire x1="81.15789375" y1="8.49869375" x2="86.17509375" y2="8.87696875" width="0" layer="19" extent="16-16"/>
+<wire x1="79.9084" y1="5.842" x2="78.935959375" y2="8.443184375" width="0" layer="19" extent="1-1"/>
+<wire x1="76.428890625" y1="2.80698125" x2="76.75815625" y2="5.46556875" width="0" layer="19" extent="16-16"/>
+<wire x1="71.718440625" y1="8.44644375" x2="76.75815625" y2="5.46556875" width="0" layer="19" extent="16-16"/>
+<wire x1="58.166" y1="7.608" x2="66.06786875" y2="7.0846875" width="0" layer="19" extent="16-16"/>
+<wire x1="53.9242" y1="1.9177" x2="56.87100625" y2="6.88299375" width="0" layer="19" extent="1-1"/>
+<wire x1="36.84949375" y1="2.7178" x2="53.9242" y2="1.9177" width="0" layer="19" extent="1-1"/>
+<wire x1="31.70933125" y1="-0.130890625" x2="36.84949375" y2="2.7178" width="0" layer="19" extent="1-1"/>
+<wire x1="9.779" y1="3.302" x2="17.78" y2="0" width="0" layer="19" extent="1-1"/>
+<wire x1="3.29" y1="-7.62" x2="9.144" y2="1.524" width="0" layer="19" extent="1-1"/>
 </signal>
 <signal name="N$54">
@@
 <wire x1="71.424275" y1="7.556840625" x2="78.041159375" y2="7.556840625" width="0.254" layer="1"/>
 <wire x1="95.085178125" y1="4.419178125" x2="97.143" y2="6.477" width="0.254" layer="16"/>
+<contactref element="C10" pad="1"/>
+<wire x1="1.79" y1="-7.62" x2="17.272" y2="7.493" width="0" layer="19" extent="1-1"/>
 </signal>
 <signal name="IT+">
@@
 <contactref element="U10" pad="3"/>
 <contactref element="U11" pad="4"/>
-<contactref element="R56" pad="2"/>
 <wire x1="81.28" y1="22.86" x2="81.15789375" y2="22.73789375" width="0.508" layer="16"/>
 <wire x1="81.15789375" y1="22.73789375" x2="81.15789375" y2="16.79869375" width="0.508" layer="16"/>
@@
 <wire x1="75.87091875" y1="70.17908125" x2="75.87091875" y2="75.814" width="0.508" layer="1"/>
 <wire x1="79.454003125" y1="70.024996875" x2="82.169" y2="67.31" width="0.508" layer="1"/>
-<wire x1="79.454003125" y1="70.024996875" x2="79.454003125" y2="70.8718" width="0.508" layer="1"/>
 <wire x1="82.169" y1="67.31" x2="83.82" y2="65.659" width="0.508" layer="1"/>
 </signal>
@@
 <contactref element="C25" pad="2"/>
 <contactref element="C1" pad="2"/>
-<contactref element="U11" pad="3"/>
 <contactref element="R33" pad="2"/>
 <contactref element="D6" pad="1"/>
 <contactref element="F2" pad="2"/>
-<contactref element="D14" pad="1"/>
 <contactref element="U$31" pad="1"/>
 <contactref element="U$31" pad="2"/>
@@
 <wire x1="109.767321875" y1="59.551" x2="108.585" y2="59.551" width="0.254" layer="1"/>
 <wire x1="83.979096875" y1="72.6041625" x2="83.979096875" y2="70.9311375" width="0.762" layer="1"/>
-<wire x1="83.979096875" y1="70.9311375" x2="84.023003125" y2="70.88723125" width="0.508" layer="1"/>
 <wire x1="122.809" y1="64.008" x2="110.236" y2="64.008" width="1.524" layer="15"/>
 <wire x1="110.236" y1="64.008" x2="106.934" y2="60.706" width="0.508" layer="15"/>
@@
 <via x="87.376" y="70.866" extent="1-16" drill="1.778"/>
 <wire x1="87.376" y1="70.866" x2="84.044234375" y2="70.866" width="0.762" layer="1"/>
-<wire x1="84.044234375" y1="70.866" x2="84.023003125" y2="70.88723125" width="0.508" layer="1"/>
 <wire x1="87.376" y1="70.866" x2="94.361" y2="77.851" width="0.508" layer="16"/>
 <wire x1="94.361" y1="77.851" x2="100.242" y2="77.851" width="0.508" layer="16"/>
@@
 <wire x1="91.694" y1="25.654" x2="90.932" y2="24.892" width="0.254" layer="1"/>
 <wire x1="90.932" y1="24.892" x2="90.932" y2="22.721" width="0.254" layer="1"/>
-<wire x1="83.69789375" y1="16.79869375" x2="83.69789375" y2="22.99189375" width="0.254" layer="16"/>
 <wire x1="83.69789375" y1="22.99189375" x2="86.741" y2="26.035" width="0.254" layer="16"/>
 <wire x1="103.74" y1="73.279" x2="103.74" y2="67.31" width="0.254" layer="1"/>
@@
 <wire x1="188.447378125" y1="57.41968125" x2="189.454596875" y2="56.4124625" width="0.254" layer="16"/>
 <wire x1="189.454596875" y1="56.4124625" x2="198.671275" y2="56.4124625" width="0.254" layer="16"/>
-</signal>
-<signal name="N$1">
-<contactref element="R56" pad="1"/>
-<contactref element="D14" pad="2"/>
-<wire x1="81.154003125" y1="70.8718" x2="81.169434375" y2="70.88723125" width="0.762" layer="1"/>
-<wire x1="81.169434375" y1="70.88723125" x2="82.373003125" y2="70.88723125" width="0.508" layer="1"/>
+<wire x1="84.044234375" y1="70.866" x2="83.979096875" y2="70.9311375" width="0" layer="19" extent="1-1"/>
 </signal>
 </signals>

Commit message: final changes
Parts:
- added C11: CAPACITOR_0603_10V_0.1UF, HyTechDevices:0603-CAP
- moved C10 72.5 mm to (73.4, 7.62), turned to 90 degrees
- moved R51 3.77 mm to (79.3, -0.24), turned to 180 degrees
Connections:
- net GND: now also C11.2
- net N$14: now also C11.1
Routing:
- net TS-FUSED: track 646.7 -> 641.5 mm
- net N$14: track 2.04 -> 7.13 mm
- net ENABLE: track 70.0 -> 66.2 mm
- net GND: track 65.0 -> 68.5 mm

Commit message: final fixes
Parts:
- R27: value RESISTOR_0805_1 -> RESISTOR_0805_12.4
Connections:
- net TS-FUSED: now also U11.3
Routing:
- net TS-FUSED: track 641.5 -> 652.0 mm
Other:
- board text added: "Tractive System Board Rev1 Designed by Cody Kaminsky 2021"
Changed lines of the file:
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@@
 <drawing>
 <settings>
-<setting alwaysvectorfont="no"/>
+<setting alwaysvectorfont="yes"/>
 <setting verticaltext="up"/>
 </settings>
@@
 <wire x1="9.200590625" y1="71.320159375" x2="16.914209375" y2="71.320159375" width="0.001" layer="120" curve="149.246308"/>
 <wire x1="9.200590625" y1="71.320159375" x2="8.13993125" y2="72.38083125" width="0.001" layer="120" style="shortdash"/>
+<text x="48.26" y="78.74" size="1.778" layer="51" rot="R90">Tractive System Board Rev1
+Designed by Cody Kaminsky 2021</text>
 </plain>
 <attributes>
@@
 <attribute name="VOLTAGE_MAX" value="150V" x="114.554" y="82.931" size="1.778" layer="27" rot="R180" display="off"/>
 </element>
-<element name="R27" library="HyTechDevices" package="0805-RES" value="RESISTOR_0805_1" x="188.722" y="17.399" smashed="yes" rot="R270">
-<attribute name="DKPN" value="P1.0DTR-ND" x="188.722" y="17.399" size="1.778" layer="27" rot="R270" display="off"/>
-<attribute name="MANUFACTURER" value="Panasonic Electronic Components" x="188.722" y="17.399" size="1.778" layer="27" rot="R270" display="off"/>
-<attribute name="MOPN" value="667-ERJ-6RQF1R0V" x="188.722" y="17.399" size="1.778" layer="27" rot="R270" display="off"/>
-<attribute name="MPN" value="ERJ-6RQF1R0V" x="188.722" y="17.399" size="1.778" layer="27" rot="R270" display="off"/>
+<element name="R27" library="HyTechDevices" package="0805-RES" value="RESISTOR_0805_12.4" x="188.722" y="17.399" smashed="yes" rot="R270">
+<attribute name="DKPN" value="P12.4CTR-ND" x="188.722" y="17.399" size="1.778" layer="27" rot="R270" display="off"/>
+<attribute name="MANUFACTURER" value="  Panasonic Electronic Components" x="188.722" y="17.399" size="1.778" layer="27" rot="R270" display="off"/>
+<attribute name="MOPN" value="667-ERJ-6ENF12R4V" x="188.722" y="17.399" size="1.778" layer="27" rot="R270" display="off"/>
+<attribute name="MPN" value="ERJ-6ENF12R4V" x="188.722" y="17.399" size="1.778" layer="27" rot="R270" display="off"/>
 <attribute name="NAME" x="189.572" y="17.399" size="0.8128" layer="25" font="vector" rot="R270" align="bottom-center"/>
-<attribute name="POWER" value="0.125W" x="188.722" y="17.399" size="1.778" layer="27" rot="R270" display="off"/>
-<attribute name="RESISTANCE" value="1" x="188.722" y="17.399" size="1.778" layer="27" rot="R270" display="off"/>
+<attribute name="POWER" value=".125W" x="188.722" y="17.399" size="1.778" layer="27" rot="R270" display="off"/>
+<attribute name="RESISTANCE" value="12.4" x="188.722" y="17.399" size="1.778" layer="27" rot="R270" display="off"/>
 <attribute name="TOLERANCE" value="1%" x="188.722" y="17.399" size="1.778" layer="27" rot="R270" display="off"/>
-<attribute name="VOLTAGE_CONTINUOUS" value="" x="188.722" y="17.399" size="1.778" layer="27" rot="R270" display="off"/>
+<attribute name="VOLTAGE_CONTINUOUS" value="1.24V" x="188.722" y="17.399" size="1.778" layer="27" rot="R270" display="off"/>
 <attribute name="VOLTAGE_MAX" value="150V" x="188.722" y="17.399" size="1.778" layer="27" rot="R270" display="off"/>
 </element>
@@
 <wire x1="87.376" y1="70.866" x2="85.717259375" y2="70.866" width="0.762" layer="1"/>
 <wire x1="85.717259375" y1="70.866" x2="83.979096875" y2="72.6041625" width="0.762" layer="1"/>
+<contactref element="U11" pad="3"/>
+<wire x1="83.69789375" y1="16.79869375" x2="83.69789375" y2="22.99189375" width="0.508" layer="16"/>
+<wire x1="83.69789375" y1="22.99189375" x2="86.741" y2="26.035" width="0.508" layer="16"/>
 </signal>
 </signals>
