File: EAGLE Board Designs/Tractive System Board/Tractive System Board Rev3.brd (EAGLE design)
At the start: 206.7 x 150.3 mm, 187 parts, among them J1 CONNECTOR-5_MICRO_V6S_, J2 CONNECTOR-5_MICRO_V7S_, J3 CONNECTOR-8_S_S, J5 CONNECTOR-4__, K4 RELAY_SPST_NC_POLARIZED_3550_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, K5 RELAY_SPST_NO_3550_12, Q2 TRANSISTOR_N_MOS__PMV15ENEA, U1 LTC6994-2, U10 DCM4623TD2J13D0T70, U11 RELAY_SOLIDSTATE_NC_AG, U16 LTC3639, U17 VOLTAGE_REGULATOR_ADJ_LR8_DPAK, U18 ISO224B_AIRGAP, U19 ISO224B_AIRGAP, U2 VOLTAGE_REGULATOR_SOT223_5V, U3 LTC6994-2

Commit message: Finished board design
Parts:
- R1, R10: value RESISTOR_0603_360K -> RESISTOR_0603_HV750K
- R6, R7, R8, R9: value RESISTOR_0603_33K -> RESISTOR_0603_HV75K
