File: EAGLE Board Designs/Tractive System Board/Tractive System Board Rev3.sch (EAGLE design)
At the start: 137 parts, among them J1 CONNECTOR-5_MICRO_V6S_, J2 CONNECTOR-5_MICRO_V7S_, J3 CONNECTOR-8_S_S, J5 CONNECTOR-4__, K4 RELAY_SPST_NC_POLARIZED_3550_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, K5 RELAY_SPST_NO_3550_12, Q2 TRANSISTOR_N_MOS__PMV15ENEA, U1 LTC6994-2, U10 DCM4623TD2J13D0T70, U11 RELAY_SOLIDSTATE_NC_AG, U16 LTC3639, U17 VOLTAGE_REGULATOR_ADJ_LR8_DPAK, U18 ISO224B_AIRGAP, U19 ISO224B_AIRGAP, U2 VOLTAGE_REGULATOR_SOT223_5V, U3 LTC6994-2

Commit message: Finished board design
Parts:
- R1, R10: value RESISTOR_0603_360K -> RESISTOR_0603_HV750K; device HyTechDevices:RESISTOR_0603_360K -> HyTechDevices:RESISTOR_0603_HV750K
- R6, R7, R8, R9: value RESISTOR_0603_33K -> RESISTOR_0603_HV75K; device HyTechDevices:RESISTOR_0603_33K -> HyTechDevices:RESISTOR_0603_HV75K
Changed lines of the file:
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@@
 <part name="C10" library="HyTechDevices" deviceset="CAPACITOR_?_*" device="0603" technology="10V_0.1UF"/>
 <part name="U$29" library="HyTechSupplies" deviceset="TS-FUSED" device=""/>
-<part name="R1" library="HyTechDevices" deviceset="RESISTOR_?_*" device="0603" technology="360K"/>
+<part name="R1" library="HyTechDevices" deviceset="RESISTOR_?_*" device="0603" technology="HV750K" value="RESISTOR_0603_HV750K"/>
 <part name="R2" library="HyTechDevices" deviceset="RESISTOR_?_*" device="0603" technology="510K"/>
-<part name="R6" library="HyTechDevices" deviceset="RESISTOR_?_*" device="0603" technology="33K"/>
-<part name="R7" library="HyTechDevices" deviceset="RESISTOR_?_*" device="0603" technology="33K"/>
-<part name="R8" library="HyTechDevices" deviceset="RESISTOR_?_*" device="0603" technology="33K"/>
-<part name="R9" library="HyTechDevices" deviceset="RESISTOR_?_*" device="0603" technology="33K"/>
-<part name="R10" library="HyTechDevices" deviceset="RESISTOR_?_*" device="0603" technology="360K"/>
+<part name="R6" library="HyTechDevices" deviceset="RESISTOR_?_*" device="0603" technology="HV75K" value="RESISTOR_0603_HV75K"/>
+<part name="R7" library="HyTechDevices" deviceset="RESISTOR_?_*" device="0603" technology="HV75K" value="RESISTOR_0603_HV75K"/>
+<part name="R8" library="HyTechDevices" deviceset="RESISTOR_?_*" device="0603" technology="HV75K" value="RESISTOR_0603_HV75K"/>
+<part name="R9" library="HyTechDevices" deviceset="RESISTOR_?_*" device="0603" technology="HV75K" value="RESISTOR_0603_HV75K"/>
+<part name="R10" library="HyTechDevices" deviceset="RESISTOR_?_*" device="0603" technology="HV750K" value="RESISTOR_0603_HV750K"/>
 <part name="R11" library="HyTechDevices" deviceset="RESISTOR_?_*" device="0603" technology="510K"/>
 <part name="XF1" library="HyTechDevices" deviceset="FUSE_HOLDER_*" device="PTH" technology="MINIBLADE"/>

Commit message: Made specified changes to the tsb
Parts:
- removed RV1: 1M, HyTechDevices:RESISTOR_0805_1M
- removed U$1: RELAY_SOLIDSTATE_NO, HyTechDevices:RELAY_SOLIDSTATE_NO
- added K1: RELAY_SOLIDSTATE_NO_AG, HyTechDevicesTempTSB:RELAY_SOLIDSTATE_NO_AG
- added R14: RESISTOR_0805_523K, HyTechDevices:RESISTOR_0805_523K
- added TP17, TP21, TP22: TEST_POINT, HyTechDevices:TEST_POINT
- R11, R2: value RESISTOR_0603_510K -> RESISTOR_0603_360K; device HyTechDevices:RESISTOR_0603_510K -> HyTechDevices:RESISTOR_0603_360K
- R12, R13: value RESISTOR_0603_510K -> RESISTOR_0603_75K; device HyTechDevices:RESISTOR_0603_510K -> HyTechDevices:RESISTOR_0603_75K
- R15: value 523k -> RESISTOR_0805_1M
- R26, R27: value RESISTOR_0603_3.3 -> RESISTOR_0603_39; device HyTechDevices:RESISTOR_0603_3.3 -> HyTechDevices:RESISTOR_0603_39
- R3: value RESISTOR_0603_8.66K -> RESISTOR_0603_8.35K; device HyTechDevices:RESISTOR_0603_8.66K -> HyTechDevices:RESISTOR_0603_8.35K
- R4: value RESISTOR_0603_13K -> RESISTOR_0603_13.3K; device HyTechDevices:RESISTOR_0603_13K -> HyTechDevices:RESISTOR_0603_13.3K
- R44: value RESISTOR_0805_1M -> RESISTOR_0805_523K; device HyTechDevices:RESISTOR_0805_1M -> HyTechDevices:RESISTOR_0805_523K
- R46: value RESISTOR_0805_523K -> RESISTOR_0805_1M; device HyTechDevices:RESISTOR_0805_523K -> HyTechDevices:RESISTOR_0805_1M
- R63: value RESISTOR_0603_1K -> RESISTOR_0603_180; device HyTechDevices:RESISTOR_0603_1K -> HyTechDevices:RESISTOR_0603_180
- renumbered RV2 to R15, U11 to K2
Connections:
- removed net N$13: R11.1, R49.1, R8.2, R9.2
- removed net N$23: R2.1, R50.1, R6.2, R7.2
- removed net N$58: C3.1, C31.1, D10.A, D14.A, R45.2, R47.1, U17.OUT
- new net LR8_O: C3.1, C31.1, D10.A, D14.A, R45.2, R47.1, TP17.P$1, U17.OUT
- new net P_DO: R11.1, R49.1, R8.2, R9.2, TP22.P$1
- new net TS_DO: R2.1, R50.1, R6.2, R7.2, TP21.P$1
- net GND: now also K1.CONTROL-; no longer U$1.CONTROL-
- net N$10: now also R14.2; no longer RV1.2
- net N$53: now also K1.CONTROL+; no longer U$1.CONTROL+
- net N$57: now also K1.CONTACT1; no longer U$1.CONTACT1
- net N$9: now also R14.1; no longer RV1.1
- net PACK+: now also K1.CONTACT2; no longer U$1.CONTACT2
Other:
- note added: "Overvoltage: 145V Undervoltage: 56V"
- note added: "Shunt resistor rated to 50 mA"
- note removed: "Overvoltage: 140V Undervoltage: 56V"
- note removed: "Shunt resistor rated to 174 mA"
