File: ESF Schematics/2022/Accumulator TS Schematic.sch (EAGLE design)
At the start: 73 parts, among them J1 CONNECTOR-1_LCAX2-14F-E, J2 CONNECTOR-1_LCAX2-14F-E, J3 CONNECTOR-1_LCAX2-14F-E, J4 CONNECTOR-1_LCAX2-14F-E, J5 CONNECTOR-1_CT2242-2, J6 CONNECTOR-5_MICROFIT, J7 CONNECTOR-1_CT2242-2, J8 CONNECTOR-5_MICROFIT

Commit message: more changes
Parts:
- PRECHARGE_RES: value 1.5k -> 7.5k
Other:
- note removed: "Add HVD panduits-done fix resistor dividers-done fix busbar labelling and gauges-done rename relay_ctrl as precharge_ok-done fix maintenance plug symbol-done fix TSMPs add isolation for DCDC-done prechargeOK same as relay_ctrl-done show all microfit connectors-done ring terminals between fused and unfused and pack plus-done"
- moved on the sheet: F1
Changed lines of the file:
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@@
 <setting verticaltext="up"/>
 </settings>
-<grid distance="0.1" unitdist="inch" unit="inch" style="lines" multiple="1" display="no" altdistance="0.01" altunitdist="inch" altunit="inch"/>
+<grid distance="0.1" unitdist="inch" unit="inch" style="lines" multiple="1" display="yes" altdistance="0.01" altunitdist="inch" altunit="inch"/>
 <layers>
 <layer number="1" name="Top" color="4" fill="1" visible="no" active="no"/>
@@
 <part name="P2" library="HyTechSupplies" deviceset="GND" device=""/>
 <part name="P3" library="HyTechSupplies" deviceset="GND" device=""/>
-<part name="PRECHARGE_RES" library="HyTechDevices" deviceset="RESISTOR_VALUE" device="" value="1.5k"/>
+<part name="PRECHARGE_RES" library="HyTechDevices" deviceset="RESISTOR_VALUE" device="" value="7.5k"/>
 <part name="P4" library="HyTechSupplies" deviceset="TS+UNFUSED" device=""/>
 <part name="TSMP-RES" library="HyTechDevices" deviceset="RESISTOR_VALUE" device="" value="10K"/>
@@
 <attribute name="DESCRIPTION_1" value="ESF compliant representation of the accumulator "/>
 <attribute name="DESCRIPTION_2" value="internals"/>
+<attribute name="DESIGNER_SCHEMATIC" value="Zekun Li"/>
 <attribute name="ENGINEER" value="Zekun Li"/>
+<attribute name="REVIEWER_SCHEMATIC" value="Arvind Srinivasan"/>
 </part>
 <part name="P12" library="HyTechSupplies" deviceset="GND" device=""/>
@@
 <text x="160.02" y="76.2" size="1.27" layer="97" align="top-left">22AWG</text>
 <text x="111.76" y="78.74" size="1.27" layer="97" align="top-left">22AWG</text>
-<text x="93.98" y="76.2" size="1.27" layer="97">PCB Trace</text>
+<text x="53.34" y="76.2" size="1.27" layer="97" rot="MR0">PCB Trace</text>
 <text x="83.82" y="175.26" size="1.27" layer="97" align="top-left">17.5mm^2</text>
 <text x="195.58" y="175.26" size="1.27" layer="97" align="top-left">PCB Trace</text>
@@
 <text x="121.92" y="205.74" size="1.27" layer="97" align="top-left">22AWG</text>
 <text x="88.9" y="198.12" size="1.27" layer="97" align="top-left">22AWG</text>
-<text x="43.18" y="76.2" size="1.27" layer="97" align="top-left">16AWG</text>
-<text x="299.72" y="187.96" size="1.778" layer="88" align="top-left">Add HVD panduits-done
-fix resistor dividers-done
-fix busbar labelling and gauges-done
-rename relay_ctrl as precharge_ok-done
-fix maintenance plug symbol-done
-fix TSMPs
-add isolation for DCDC-done
-prechargeOK same as relay_ctrl-done
-show all microfit connectors-done
-ring terminals between fused and unfused and pack plus-done</text>
+<text x="104.14" y="76.2" size="1.27" layer="97" rot="MR0" align="top-left">16AWG</text>
 <text x="30.48" y="119.38" size="1.27" layer="97">17.5mm^2</text>
 <text x="30.48" y="127" size="1.27" layer="97" align="top-left">17.5mm^2</text>
@@
 <text x="96.52" y="99.06" size="1.27" layer="97">PCB Trace</text>
 <text x="190.5" y="187.96" size="1.27" layer="97" align="top-left">PCB Trace</text>
+<text x="147.32" y="165.1" size="1.27" layer="97" align="top-left">PCB Trace</text>
+<text x="7.62" y="137.16" size="1.27" layer="97" align="top-left">22AWG</text>
 </plain>
 <instances>
 <instance part="U$1" gate="G$1" x="152.4" y="81.28" smashed="yes" rot="MR0"/>
-<instance part="U$2" gate="G$1" x="88.9" y="81.28" smashed="yes" rot="MR0"/>
+<instance part="U$2" gate="G$1" x="58.42" y="81.28" smashed="yes"/>
 <instance part="U$3" gate="G$1" x="88.9" y="144.78" smashed="yes" rot="R90"/>
 <instance part="U$4" gate="G$1" x="101.6" y="144.78" smashed="yes" rot="R90"/>
@@
 </instance>
 <instance part="U$14" gate="G$1" x="55.88" y="142.24" smashed="yes"/>
-<instance part="F1" gate="G$1" x="55.88" y="78.74" smashed="yes">
-<attribute name="NAME" x="54.61" y="80.01" size="1.27" layer="95" align="bottom-center"/>
-<attribute name="VALUE" x="54.61" y="77.47" size="1.27" layer="96" align="top-center"/>
+<instance part="F1" gate="G$1" x="91.44" y="78.74" smashed="yes" rot="MR0">
+<attribute name="NAME" x="92.71" y="80.01" size="1.27" layer="95" rot="MR0" align="bottom-center"/>
+<attribute name="VALUE" x="92.71" y="77.47" size="1.27" layer="96" rot="MR0" align="top-center"/>
 </instance>
 <instance part="P8" gate="1" x="157.48" y="81.28" smashed="yes">
@@
 <attribute name="VALUE" x="10.16" y="129.54" size="1.27" layer="96" align="top-center"/>
 </instance>
-<instance part="U$21" gate="G$1" x="93.98" y="68.58" smashed="yes">
-<attribute name="VALUE" x="93.98" y="66.04" size="1.27" layer="96" align="top-center"/>
-</instance>
-<instance part="U$22" gate="G$1" x="93.98" y="81.28" smashed="yes">
-<attribute name="VALUE" x="93.98" y="86.36" size="1.27" layer="96" align="bottom-center"/>
+<instance part="U$21" gate="G$1" x="53.34" y="68.58" smashed="yes" rot="MR0">
+<attribute name="VALUE" x="53.34" y="66.04" size="1.27" layer="96" rot="MR0" align="top-center"/>
+</instance>
+<instance part="U$22" gate="G$1" x="53.34" y="81.28" smashed="yes" rot="MR0">
+<attribute name="VALUE" x="53.34" y="86.36" size="1.27" layer="96" rot="MR0" align="bottom-center"/>
 </instance>
 <instance part="U$23" gate="G$1" x="119.38" y="81.28" smashed="yes">
@@
 <segment>
 <pinref part="U$2" gate="G$1" pin="-IN"/>
-<wire x1="91.44" y1="71.12" x2="93.98" y2="71.12" width="0.0762" layer="91"/>
+<wire x1="55.88" y1="71.12" x2="53.34" y2="71.12" width="0.0762" layer="91"/>
 <pinref part="U$21" gate="G$1" pin="TS-UNFUSED"/>
 </segment>
@@
 <segment>
 <pinref part="U$2" gate="G$1" pin="+OUT"/>
-<wire x1="60.96" y1="78.74" x2="58.42" y2="78.74" width="0.254" layer="91"/>
+<wire x1="86.36" y1="78.74" x2="88.9" y2="78.74" width="0.254" layer="91"/>
 <pinref part="F1" gate="G$1" pin="2"/>
 </segment>
@@
 <segment>
 <pinref part="U$2" gate="G$1" pin="-OUT"/>
-<wire x1="60.96" y1="71.12" x2="58.42" y2="71.12" width="0.254" layer="91"/>
-<label x="58.42" y="71.12" size="1.27" layer="95" rot="R180" xref="yes"/>
+<wire x1="86.36" y1="71.12" x2="88.9" y2="71.12" width="0.254" layer="91"/>
+<label x="88.9" y="71.12" size="1.27" layer="95" rot="MR180" xref="yes"/>
 </segment>
 </net>
@@
 <segment>
 <pinref part="F1" gate="G$1" pin="1"/>
-<wire x1="50.8" y1="78.74" x2="48.26" y2="78.74" width="0.254" layer="91"/>
-<label x="48.26" y="78.74" size="1.27" layer="95" rot="R180" xref="yes"/>
+<wire x1="96.52" y1="78.74" x2="99.06" y2="78.74" width="0.254" layer="91"/>
+<label x="99.06" y="78.74" size="1.27" layer="95" rot="MR180" xref="yes"/>
 </segment>
 </net>
@@
 <segment>
 <pinref part="U$2" gate="G$1" pin="+IN"/>
-<wire x1="91.44" y1="78.74" x2="93.98" y2="78.74" width="0.0762" layer="91"/>
+<wire x1="55.88" y1="78.74" x2="53.34" y2="78.74" width="0.0762" layer="91"/>
 <pinref part="U$22" gate="G$1" pin="TS+"/>
 </segment>

Commit message: yet more fixes in preparation for submission
Parts:
- removed U$12: LOGICGATE_INVERTER, HyTechSymbolsTemp:LOGICGATE_INVERTER
- removed U$13: MOSFET_N-CHANNEL, HyTechSymbolsTemp:MOSFET_N-CHANNEL
Connections:
- net OKHS renamed IMD_OK
- removed net N$11: U$12.!IN, U$13.G
- removed net N$13: PRECHARGE.COIL+, U$13.D
- net GND: no longer U$13.S
- net PRECHARGE_OK: now also PRECHARGE.COIL+; no longer U$12.IN
Changed lines of the file:
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@@
 <setting verticaltext="up"/>
 </settings>
-<grid distance="0.1" unitdist="inch" unit="inch" style="lines" multiple="1" display="yes" altdistance="0.01" altunitdist="inch" altunit="inch"/>
+<grid distance="0.1" unitdist="inch" unit="inch" style="lines" multiple="1" display="no" altdistance="0.01" altunitdist="inch" altunit="inch"/>
 <layers>
 <layer number="1" name="Top" color="4" fill="1" visible="no" active="no"/>
@@
 <part name="P1" library="HyTechSupplies" deviceset="GND" device=""/>
 <part name="PRECHARGE" library="HyTechSymbolsTemp" deviceset="RELAY_SPST_NO_?*" device="" technology="3350-1275-126"/>
-<part name="U$12" library="HyTechSymbolsTemp" deviceset="LOGICGATE_INVERTER" device=""/>
-<part name="U$13" library="HyTechSymbolsTemp" deviceset="MOSFET_N-CHANNEL" device=""/>
-<part name="P2" library="HyTechSupplies" deviceset="GND" device=""/>
 <part name="P3" library="HyTechSupplies" deviceset="GND" device=""/>
 <part name="PRECHARGE_RES" library="HyTechDevices" deviceset="RESISTOR_VALUE" device="" value="7.5k"/>
@@
 <text x="104.14" y="142.24" size="1.27" layer="97">17.5mm^2</text>
 <text x="88.9" y="142.24" size="1.27" layer="97">17.5mm^2</text>
-<text x="55.88" y="111.76" size="1.27" layer="97" align="top-left">PCB Trace</text>
+<text x="60.96" y="111.76" size="1.27" layer="97" align="top-left">PCB Trace</text>
 <text x="40.64" y="142.24" size="1.27" layer="97" align="top-left">22AWG</text>
 <text x="35.56" y="162.56" size="1.27" layer="97" align="top-left">22AWG</text>
@@
 <attribute name="NAME" x="71.12" y="117.602" size="1.27" layer="95"/>
 </instance>
-<instance part="U$12" gate="G$1" x="30.48" y="101.6" smashed="yes"/>
-<instance part="U$13" gate="G$1" x="45.72" y="104.14" smashed="yes">
-<attribute name="NAME" x="45.72" y="109.22" size="1.27" layer="95" align="bottom-center"/>
-</instance>
-<instance part="P2" gate="1" x="50.8" y="93.98" smashed="yes">
-<attribute name="VALUE" x="50.8" y="92.71" size="1.27" layer="96" align="top-center"/>
-</instance>
 <instance part="P3" gate="1" x="152.4" y="160.02" smashed="yes">
 <attribute name="VALUE" x="152.4" y="158.75" size="1.27" layer="96" align="top-center"/>
@@
 </segment>
 <segment>
-<pinref part="U$13" gate="G$1" pin="S"/>
-<wire x1="50.8" y1="99.06" x2="50.8" y2="96.52" width="0.0762" layer="91"/>
-<pinref part="P2" gate="1" pin="GND"/>
-</segment>
-<segment>
 <pinref part="AIR-" gate="G$1" pin="COIL+"/>
 <wire x1="154.94" y1="162.56" x2="152.4" y2="162.56" width="0.1524" layer="91"/>
@@
 <net name="PRECHARGE_OK" class="0">
 <segment>
-<pinref part="U$12" gate="G$1" pin="IN"/>
-<wire x1="27.94" y1="101.6" x2="25.4" y2="101.6" width="0.0762" layer="91"/>
-<label x="25.4" y="101.6" size="1.27" layer="95" rot="R180" xref="yes"/>
-</segment>
-<segment>
 <pinref part="U$30" gate="G$1" pin="PRECHARGE_OK"/>
 <wire x1="251.46" y1="119.38" x2="254" y2="119.38" width="0.0762" layer="91"/>
@@
 <wire x1="68.58" y1="177.8" x2="68.58" y2="162.56" width="0.0762" layer="91"/>
 </segment>
-</net>
-<net name="N$11" class="0">
-<segment>
-<pinref part="U$12" gate="G$1" pin="!IN"/>
-<pinref part="U$13" gate="G$1" pin="G"/>
-<wire x1="39.37" y1="101.6" x2="40.64" y2="101.6" width="0.0762" layer="91"/>
-</segment>
-</net>
-<net name="N$13" class="0">
-<segment>
-<pinref part="U$13" gate="G$1" pin="D"/>
+<segment>
 <pinref part="PRECHARGE" gate="G$1" pin="COIL+"/>
-<wire x1="50.8" y1="109.22" x2="68.58" y2="109.22" width="0.0762" layer="91"/>
+<wire x1="68.58" y1="109.22" x2="60.96" y2="109.22" width="0.1524" layer="91"/>
+<label x="60.96" y="109.22" size="1.27" layer="95" rot="R180" xref="yes"/>
 </segment>
 </net>
@@
 </segment>
 </net>
-<net name="OKHS" class="0">
+<net name="IMD_OK" class="0">
 <segment>
 <pinref part="U$1" gate="G$1" pin="OKHS"/>
