File: ESF Schematics/2022/Charging Shutdown Circuit Schematic.sch (EAGLE design)
At the start: 27 parts, among them J1 CONNECTOR-2_HPK, J2 CONNECTOR-2_HPK, J3 CONNECTOR-1_LCAX2-14F-E, J4 CONNECTOR-1_LCAX2-14F-E, J5 CONNECTOR-1_LCAX2-14F-E, J6 CONNECTOR-1_LCAX2-14F-E, J7 CONNECTOR-3_NEMA-5-15, J8 CONNECTOR-3_HV02-M3S(40A), J9 CONNECTOR-3_HV02-M3S(40A)

Commit message: fixups after the ESF review
Parts:
- added F1: 3A, HyTechSymbolsTemp:FUSE
- added J10, J11, J12, J13: CONNECTOR-1_LCAX2-14F-E, HyTechSymbolsTemp:CONNECTOR-1_LCAX2-14F-E
- added U$11: CHARGER_CONTROLLER, HyTechSymbolsTemp:CHARGER_CONTROLLER
- added U$12: BENDER_IR155-3204, HyTechSymbols:BENDER_IR155-3204
Connections:
- new net +12V: F1.1, U$12.+12V
- new net HVD+: J10.1
- new net HVD-: J11.1
- new net N$14: AIR2.CONTACT2, J12.1
- new net N$6: F1.2, IMD_RELAY.6
- new net OKHS: U$12.OKHS
- new net TS+: U$12.XLA+(HV+)
- new net TS-UNFUSED: U$12.XLA-(HV-)
- net CHARGER_CONTROLLER_CANH: now also U$11.CANH
- net CHARGER_CONTROLLER_CANL: now also U$11.CANL
- net GND: now also U$12.GND
- net N$13: now also J13.1; no longer AIR2.CONTACT2
Other:
- note added: "(>= 6 mil)"
- note added: "(Busbar)"
- note added: "HVD connectors-done busbar labelling-done add PS to relay for shdn-done charger controller box-done move interlocks outside accumulator-done"
- note added: "PCB Trace"
- note added: "PCB Trace:"
- note removed: "HVD connectors busbar labelling add PS to relay for shdn charger controller box move interlocks outside accumulator"
- moved on the sheet: HPK_INTERLOCK, HVD_INTERLOCK

Commit message: more changes
Parts:
- added J14, J15: CONNECTOR-3_NEMA-5-20, HyTechSymbolsTemp:CONNECTOR-3_NEMA-5-20
- added U$15: INLINE_GFCI, HyTechSymbolsTemp:INLINE_GFCI
- J7: value CONNECTOR-3_NEMA-5-15 -> CONNECTOR-3_NEMA-5-20; device HyTechSymbolsTemp:CONNECTOR-3_NEMA-5-15 -> HyTechSymbolsTemp:CONNECTOR-3_NEMA-5-20
- U$9: value POWER_RELAY -> REMOTE_POWER_CONTROL; device HyTechSymbolsTemp:POWER_RELAY -> HyTechSymbolsTemp:REMOTE_POWER_CONTROL
Connections:
- new net N$15: J9.3, U$9.HOT_OUT
- new net N$26: J14.1, U$15.HOT_OUT
- new net N$34: J14.3, U$15.GND_OUT
- new net N$35: J15.3, U$15.GND_IN
- new net N$36: J15.2, U$15.NEUTRAL_IN
- new net N$37: J15.1, U$15.HOTIN
- net N$31: now also J14.2, U$15.NEUTRAL_OUT; no longer J9.3, U$9.GND_OUT
- net N$33: now also U$9.GND_OUT; no longer U$9.HOT_OUT
Other:
- note added: "(>= 20 mil)"
- note added: "12AWG"
- note added: "12AWG:"
- note added: "To external AC Power"
- note removed: "(>= 6 mil)"

Commit message: yet more fixes in preparation for submission
Parts:
- U$15: value INLINE_GFCI -> REMOTE_POWER_CONTROL_RPC-20-SCD; device HyTechSymbolsTemp:INLINE_GFCI -> HyTechSymbolsTemp:REMOTE_POWER_CONTROL_RPC-20-SCD
- U$9: value REMOTE_POWER_CONTROL -> INLINE_GFCI_GFM20-3WC; device HyTechSymbolsTemp:REMOTE_POWER_CONTROL -> HyTechSymbolsTemp:INLINE_GFCI_GFM20-3WC
- renumbered AIR1 to AIR+, AIR2 to AIR-
Connections:
- removed net OKHS: U$12.OKHS
- removed net RELAY_CTRL: AIR+.COIL-, U$7.RELAY_CTRL
- new net PRECHARGE_OK: AIR+.COIL-, U$7.PRECHARGE_OK
- net IMD_OK: now also U$12.OKHS
- net N$15: now also U$15.HOT_OUT; no longer U$9.HOT_OUT
- net N$23: now also U$15.HOTIN; no longer U$9.HOTIN
- net N$24: now also U$15.NEUTRAL_IN; no longer U$9.NEUTRAL_IN
- net N$25: now also U$15.GND_IN; no longer U$9.GND_IN
- net N$26: now also U$9.HOT_OUT; no longer U$15.HOT_OUT
- net N$31: now also U$9.NEUTRAL_OUT; no longer U$15.NEUTRAL_OUT
- net N$32: now also U$15.NEUTRAL_OUT; no longer U$9.NEUTRAL_OUT
- net N$33: now also U$15.GND_OUT; no longer U$9.GND_OUT
- net N$34: now also U$9.GND_OUT; no longer U$15.GND_OUT
- net N$35: now also U$9.GND_IN; no longer U$15.GND_IN
- net N$36: now also U$9.NEUTRAL_IN; no longer U$15.NEUTRAL_IN
- net N$37: now also U$9.HOTIN; no longer U$15.HOTIN
- net SHDN: now also U$15.EN; no longer U$9.EN
Other:
- note removed: "HVD connectors-done busbar labelling-done add PS to relay for shdn-done charger controller box-done move interlocks outside accumulator-done"
