File: EAGLE Board Designs/AMS/AMS Segment/BMS Segment rev15.sch (EAGLE design)
At the start: 119 parts, among them J1_A 0R, J1_B 0R, J2_A 0R, J2_B 0R, J3_A 0R, J3_B 0R, J4_A 0R, J4_B 0R, J5_A 0R, J5_B 0R, J6_A 0R, J6_B 0R, J7_A 0R, J7_B 0R, J8_A 0R, J8_B 0R, Q1 NSV1C201MZ4, Q2 NSV1C201MZ4, U1 LTC6811-2, U2 LTC6811-2

Commit message: Cleanup (#27)
Parts:
- removed AMS_CELL_TEST: AMS_CELL_TEST, HyTechDevices:CONNECTOR-2NANO-FIT_VERTICAL-2
- removed AMS_THERM_TEST: AMS_THERM_TEST, HyTechDevices:CONNECTOR-2NANO-FIT_VERTICAL-2
- renumbered TRANSFORMER to T1, U$28 to TP2, U$29 to TP3, U$5 to TP4, U$6 to TP5, U$7 to TP6, U$8 to TP1
Connections:
- removed net SENSE17_PRE: AMS_CELL_TEST-1.S, F17.2, J_CELL_A.1
- new net CELL+: Q1.S
- new net GATE: Q1.G
- new net N$44: F17.2, J_CELL_A.1
- net GPIO3_A_POST: no longer AMS_THERM_TEST-2.S
- net GPIO3_A_PRE: no longer AMS_THERM_TEST-1.S
- net N$1: now also Q1.D
- net SENSE17_POST: no longer AMS_CELL_TEST-2.S
