File: EAGLE Board Designs/AMS/AMS Segment/AMS Segment rev18.brd (EAGLE design)
At the start: 275.2 x 86 mm, 343 parts, among them J1 CONNECTOR-2_MICROFIT_SMD_RIGH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, J10 CONNECTOR-2_MICROFIT_SMD_RIGH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, J100 CONNECTOR-1_5222_, J101 CONNECTOR-1_5222_, J102 CONNECTOR-1_5222_, J103 CONNECTOR-1_5222_, J104 CONNECTOR-1_5222_, J105 CONNECTOR-1_5222_, J106 CONNECTOR-1_5222_, J107 CONNECTOR-1_5222_, J108 CONNECTOR-1_5222_, J109 CONNECTOR-1_5222_, J110 CONNECTOR-1_5222_, J111 CONNECTOR-1_5222_, J112 CONNECTOR-1_5222_, J113 CONNECTOR-1_5222_, J114 CONNECTOR-1_5222_, J115 CONNECTOR-1_5222_, J116 CONNECTOR-1_5222_, J117 CONNECTOR-1_5222_, J118 CONNECTOR-1_5222_, J119 CONNECTOR-1_5222_, J120 CONNECTOR-1_5222_, J121 CONNECTOR-1_5222_, J2 CONNECTOR-2_MICROFIT_SMD_RIGH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, J3 CONNECTOR-2_MICROFIT_SMD_RIGH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, J4 CONNECTOR-2_MICROFIT_SMD_RIGH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, J5 CONNECTOR-2_MICROFIT_SMD_RIGH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, J6 CONNECTOR-2_MICROFIT_SMD_RIGH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, J7 CONNECTOR-2_MICROFIT_SMD_RIGH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, J8 CONNECTOR-2_MICROFIT_SMD_RIGH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, J9 CONNECTOR-2_MICROFIT_SMD_RIGH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, T1 TRANSFORMER_HM2112ZNLT, U1 SHT31-ARP-B, U2 LTC6811-2, U3 LT3990-5, U4 LT3990-5, U5 LTC6811-2, U6 SHT31-ARP-B

Commit message: Fixed silkscreen
Parts:
- added U$34: (no value), HyTechAesthetics:HV_0.50"
- moved U$32 66.1 mm to (195.6, -13.7)
- moved D2 5.08 mm to (160.7, -84.1)
- moved R21 5.08 mm to (163.8, -84.1)
- moved D3 5.08 mm to (113.2, -84.1)
- moved R32 5.08 mm to (110.1, -84.1)
- moved U$29 5.08 mm to (267.5, -9.91)
- moved U$27 3.81 mm to (20.6, -14.0)
- moved U$28 1.27 mm to (63.0, -78.7)
- moved R1 1.27 mm to (266.3, -36.8)
Routing:
- net VREGU: track 294.3 -> 289.2 mm
- net VREGL: track 265.9 -> 260.8 mm
- net N$81: track 2.10 -> 3.41 mm
- net GPIO5L: track 84.0 -> 84.5 mm
Other:
- board text added: "HyTech Racing 2022 AMS Segment rev18 Designed by Cody Kaminsky, Noah Bruckner, and Ethan Weinstock Based on rev15 by Arvind Srinivasan"
- board text removed: "HyTech Racing 2022 AMS Segment rev17 Designed by Cody Kaminsky, Noah Bruckner, and Ethan Weinstock Based on rev15 by Arvind Srinivasan"

Commit message: Fixed routing
Routing:
- net GPIO3U: track 58.0 -> 56.5 mm, vias 4 -> 2
Changed lines of the file:
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@@
 <layers>
 <layer number="1" name="Top" color="4" fill="1" visible="yes" active="yes"/>
-<layer number="2" name="Route2" color="16" fill="1" visible="no" active="yes"/>
+<layer number="2" name="Route2" color="16" fill="1" visible="yes" active="yes"/>
 <layer number="3" name="Route3" color="17" fill="1" visible="no" active="no"/>
 <layer number="4" name="Route4" color="18" fill="1" visible="no" active="no"/>
@@
 <layer number="13" name="Route13" color="21" fill="1" visible="no" active="no"/>
 <layer number="14" name="Route14" color="22" fill="1" visible="no" active="no"/>
-<layer number="15" name="Route15" color="23" fill="1" visible="no" active="yes"/>
-<layer number="16" name="Bottom" color="1" fill="1" visible="no" active="yes"/>
+<layer number="15" name="Route15" color="23" fill="1" visible="yes" active="yes"/>
+<layer number="16" name="Bottom" color="1" fill="1" visible="yes" active="yes"/>
 <layer number="17" name="Pads" color="2" fill="1" visible="yes" active="yes"/>
 <layer number="18" name="Vias" color="2" fill="1" visible="yes" active="yes"/>
@@
 <layer number="20" name="Dimension" color="24" fill="1" visible="yes" active="yes"/>
 <layer number="21" name="tPlace" color="7" fill="1" visible="yes" active="yes"/>
-<layer number="22" name="bPlace" color="7" fill="1" visible="no" active="yes"/>
+<layer number="22" name="bPlace" color="7" fill="1" visible="yes" active="yes"/>
 <layer number="23" name="tOrigins" color="15" fill="1" visible="yes" active="yes"/>
-<layer number="24" name="bOrigins" color="15" fill="1" visible="no" active="yes"/>
+<layer number="24" name="bOrigins" color="15" fill="1" visible="yes" active="yes"/>
 <layer number="25" name="tNames" color="7" fill="1" visible="yes" active="yes"/>
-<layer number="26" name="bNames" color="7" fill="1" visible="no" active="yes"/>
-<layer number="27" name="tValues" color="7" fill="1" visible="no" active="yes"/>
-<layer number="28" name="bValues" color="7" fill="1" visible="no" active="yes"/>
+<layer number="26" name="bNames" color="7" fill="1" visible="yes" active="yes"/>
+<layer number="27" name="tValues" color="7" fill="1" visible="yes" active="yes"/>
+<layer number="28" name="bValues" color="7" fill="1" visible="yes" active="yes"/>
 <layer number="29" name="tStop" color="7" fill="3" visible="no" active="yes"/>
 <layer number="30" name="bStop" color="7" fill="6" visible="no" active="yes"/>
@@
 <layer number="38" name="bTest" color="7" fill="1" visible="no" active="yes"/>
 <layer number="39" name="tKeepout" color="4" fill="11" visible="yes" active="yes"/>
-<layer number="40" name="bKeepout" color="1" fill="11" visible="no" active="yes"/>
-<layer number="41" name="tRestrict" color="4" fill="10" visible="yes" active="yes"/>
+<layer number="40" name="bKeepout" color="1" fill="11" visible="yes" active="yes"/>
+<layer number="41" name="tRestrict" color="4" fill="10" visible="no" active="yes"/>
 <layer number="42" name="bRestrict" color="1" fill="10" visible="no" active="yes"/>
 <layer number="43" name="vRestrict" color="2" fill="10" visible="no" active="yes"/>
@@
 <layer number="50" name="dxf" color="7" fill="1" visible="no" active="yes"/>
 <layer number="51" name="tDocu" color="7" fill="1" visible="yes" active="yes"/>
-<layer number="52" name="bDocu" color="7" fill="1" visible="no" active="yes"/>
+<layer number="52" name="bDocu" color="7" fill="1" visible="yes" active="yes"/>
 <layer number="53" name="tGND_GNDA" color="7" fill="9" visible="no" active="no"/>
 <layer number="54" name="bGND_GNDA" color="1" fill="9" visible="no" active="no"/>
@@
 <wire x1="69.53386875" y1="-54.155925" x2="69.53386875" y2="-53.848" width="0.1524" layer="1"/>
 <wire x1="70.47054375" y1="-55.0926" x2="71.9546875" y2="-55.0926" width="0.1524" layer="1"/>
-<wire x1="69.53386875" y1="-53.848" x2="69.215" y2="-53.848" width="0.1524" layer="15"/>
-<wire x1="69.215" y1="-53.848" x2="68.4276" y2="-53.0606" width="0.1524" layer="15"/>
-<wire x1="68.4276" y1="-53.0606" x2="68.4276" y2="-46.28970625" width="0.1524" layer="15"/>
-<wire x1="68.4276" y1="-46.28970625" x2="68.9164" y2="-45.80090625" width="0.1524" layer="15"/>
-<via x="68.9164" y="-45.80090625" extent="1-16" drill="0.254"/>
-<wire x1="70.58548125" y1="-43.79071875" x2="68.9164" y2="-45.4598" width="0.1524" layer="1"/>
-<wire x1="68.9164" y1="-45.80090625" x2="68.9164" y2="-45.4598" width="0.1524" layer="1"/>
-<wire x1="70.58548125" y1="-43.79071875" x2="70.58548125" y2="-43.02871875" width="0.1524" layer="1"/>
-<via x="70.58548125" y="-43.02871875" extent="1-16" drill="0.254"/>
-<wire x1="85.0392" y1="-28.575" x2="70.58548125" y2="-43.02871875" width="0.1524" layer="15"/>
-<wire x1="85.0392" y1="-28.575" x2="98.552" y2="-28.575" width="0.1524" layer="15"/>
 <via x="98.552" y="-28.575" extent="1-16" drill="0.254"/>
 <wire x1="102.2865" y1="-26.035" x2="102.2865" y2="-26.3932875" width="0.1524" layer="1"/>
@@
 <wire x1="100.4263" y1="-27.3232" x2="99.1745" y2="-28.575" width="0.1524" layer="1"/>
 <wire x1="98.552" y1="-28.575" x2="99.1745" y2="-28.575" width="0.1524" layer="1"/>
+<wire x1="98.552" y1="-28.575" x2="98.552" y2="-33.528" width="0.1524" layer="15"/>
+<wire x1="71.12" y1="-48.26" x2="83.82" y2="-48.26" width="0.1524" layer="15"/>
+<wire x1="98.552" y1="-33.528" x2="83.82" y2="-48.26" width="0.1524" layer="15"/>
+<wire x1="69.53386875" y1="-53.848" x2="69.53386875" y2="-52.95926875" width="0.1524" layer="15"/>
+<wire x1="69.53386875" y1="-52.95926875" x2="69.55666875" y2="-52.93646875" width="0.1524" layer="15"/>
+<wire x1="69.55666875" y1="-52.93646875" x2="69.55666875" y2="-51.16993125" width="0.1524" layer="15"/>
+<wire x1="69.55666875" y1="-51.16993125" x2="69.5285375" y2="-51.1418" width="0.1524" layer="15"/>
+<wire x1="69.5285375" y1="-51.1418" x2="69.5285375" y2="-49.8514625" width="0.1524" layer="15"/>
+<wire x1="69.5285375" y1="-49.8514625" x2="71.12" y2="-48.26" width="0.1524" layer="15"/>
 </signal>
 <signal name="N$78">
@@
 <wire x1="73.2409" y1="-8.4836" x2="73.2409" y2="-7.2651" width="0.1524" layer="1"/>
 <via x="68.99786875" y="-52.705" extent="1-16" drill="0.254"/>
-<wire x1="68.99786875" y1="-52.705" x2="68.99786875" y2="-46.80073125" width="0.1524" layer="15"/>
-<wire x1="70.2056" y1="-45.593" x2="68.99786875" y2="-46.80073125" width="0.1524" layer="15"/>
+<wire x1="68.99786875" y1="-52.705" x2="68.99786875" y2="-48.006" width="0.1524" layer="15"/>
+<wire x1="69.0626" y1="-48.006" x2="68.99786875" y2="-48.006" width="0.1524" layer="15"/>
 <wire x1="74.4474" y1="-10.7696" x2="74.4474" y2="-7.9756" width="0.1524" layer="15"/>
 <wire x1="74.4474" y1="-10.7696" x2="67.0306" y2="-18.1864" width="0.1524" layer="15"/>
@@
 <wire x1="68.99786875" y1="-52.705" x2="68.87346875" y2="-52.8294" width="0.1524" layer="1"/>
 <wire x1="68.87346875" y1="-52.8294" x2="68.87346875" y2="-54.0584375" width="0.1524" layer="1"/>
-<via x="70.2056" y="-45.593" extent="1-16" drill="0.254"/>
+<via x="69.0626" y="-48.006" extent="1-16" drill="0.254"/>
 <via x="70.381965625" y="-42.137165625" extent="1-16" drill="0.254"/>
 <wire x1="71.14428125" y1="-42.79725" x2="70.484196875" y2="-42.137165625" width="0.1524" layer="1"/>
 <wire x1="70.484196875" y1="-42.137165625" x2="70.381965625" y2="-42.137165625" width="0.1524" layer="1"/>
-<wire x1="71.14428125" y1="-44.678975" x2="70.23025625" y2="-45.593" width="0.1524" layer="1"/>
-<wire x1="70.2056" y1="-45.593" x2="70.23025625" y2="-45.593" width="0.1524" layer="1"/>
+<wire x1="71.14428125" y1="-44.678975" x2="69.0626" y2="-46.76065625" width="0.1524" layer="1"/>
+<wire x1="69.0626" y1="-48.006" x2="69.0626" y2="-46.76065625" width="0.1524" layer="1"/>
 <wire x1="71.14428125" y1="-44.678975" x2="71.14428125" y2="-42.79725" width="0.1524" layer="1"/>
 <wire x1="70.381965625" y1="-42.137165625" x2="70.357309375" y2="-42.112509375" width="0.1524" layer="15"/>

Commit message: Board fixes
Parts:
- added U$35: (no value), HyTechManufacturing:LOGO_HYTECH_EXTRA_LARGE
- U$26: device HyTechAesthetics:LOGO_HYTECH_SQUARE_EXTRA_LARGE -> HyTechManufacturing:LOGO_GT_LARGE
- moved U$26 98.4 mm to (73.0, -42.9)
- moved U$101 30.3 mm to (247.7, -42.9)
- moved U$103 26.4 mm to (28.6, -42.9)
- moved U$1 24.1 mm to (269.9, -29.8)
- moved C3 2.97 mm to (248.2, -5.08), turned to 90 degrees
- moved R3 2.87 mm to (248.2, -8.00), turned to 270 degrees
- moved F1 2.04 mm to (268.8, -17.1)
- moved F12 1.58 mm to (142.8, -33.0)
- moved U$102 1.27 mm to (115.8, -42.9)
- moved F14 0.13 mm to (113.8, -9.46)
- moved F18 0.13 mm to (51.5, -9.46)
- moved F20 0.13 mm to (42.3, -9.46)
- moved F16 0.13 mm to (81.8, -9.46)
- moved F9 0.13 mm to (204.3, -9.46)
Routing:
- net N$90: track 23.7 -> 17.4 mm
- net GPIO4L: track 75.8 -> 80.3 mm
- net V-L: track 132.4 -> 134.5 mm
- net GPIO3L: track 55.7 -> 53.6 mm
- net SENSE12: track 109.0 -> 107.3 mm
- net CC0: track 20.2 -> 19.3 mm

Commit message: Prepped rev 18 with updated lib
Parts:
- CELL10:Q1, CELL11:Q1, CELL12:Q1, CELL13:Q1, CELL14:Q1, CELL15:Q1, CELL16:Q1, CELL17:Q1, CELL18:Q1, CELL19:Q1, CELL1:Q1, CELL20:Q1, CELL21:Q1, CELL2:Q1, CELL3:Q1, CELL4:Q1, CELL5:Q1, CELL6:Q1, CELL7:Q1, CELL8:Q1, CELL9:Q1: value TRANSISTOR_P_MOS_SOT23_SI2369DS-T1-GE3 -> TRANSISTOR_P_MOS_SOT-23_SI2369DS-T1-GE3
- J100, J101, J102, J103, J104, J105, J106, J107, J108, J109, J110, J111, J112, J113, J114, J115, J116, J117, J118, J119, J120, J121: value CONNECTOR-1_5222_ -> CONNECTOR-1_5222
- TP1, TP10, TP2, TP3, TP4, TP5, TP6, TP7, TP8, TP9: device HyTechDevices:MICRO_MINIATURE -> HyTechDevices:5015
Other:
- board text removed: "DRVL"
- board text removed: "DRVU"
- board text removed: "V+L"
- board text removed: "V+U"
- board text removed: "V-L"
- board text removed: "V-U"
- board text removed: "VREGL"
- board text removed: "VREGU"
