File: EAGLE Board Designs/AMS/AMS Enerdel Adapter/BMS Enerdel Adapter rev7.brd (EAGLE design)
At the start: 329.9 x 382.3 mm, 30 parts, among them J1 CONNECTOR-1_5222_, J10 CONNECTOR-1_5222_, J11 CONNECTOR-1_5222_, J12 CONNECTOR-1_5222_, J13 CONNECTOR-1_5222_, J14 CONNECTOR-1_5222_, J15 CONNECTOR-1_5222_, J16 CONNECTOR-1_5222_, J17 CONNECTOR-1_5222_, J18 CONNECTOR-1_5222_, J19 CONNECTOR-1_5222_, J2 CONNECTOR-1_5222_, J20 CONNECTOR-1_5222_, J21 CONNECTOR-1_5222_, J22 CONNECTOR-1_5222_, J3 CONNECTOR-1_5222_, J4 CONNECTOR-1_5222_, J5 CONNECTOR-1_5222_, J6 CONNECTOR-1_5222_, J7 CONNECTOR-1_5222_, J8 CONNECTOR-1_5222_, J9 CONNECTOR-1_5222_

Commit message: Schematic Framework Finished
Parts:
- moved B-CONNECTOR-14-UPPER-IN 511.5 mm to (101.6, 369.6), turned to 270 degrees
- moved B-CONNECTOR-14-UPPER-OUT 496.8 mm to (77.5, 369.6), turned to 270 degrees
- moved A-CONNECTOR-14-UPPER-OUT 438.0 mm to (17.8, 369.6), flipped to the bottom, turned to 90 degrees
- moved A-CONNECTOR-14-UPPER-IN 433.8 mm to (41.9, 369.6), turned to 270 degrees
- moved J21 342.1 mm to (88.9, 328.9), turned to 90 degrees
- moved J19 306.0 mm to (88.9, 302.3), turned to 90 degrees
- moved J20 289.4 mm to (35.6, 304.8), turned to 90 degrees
- moved J22 280.9 mm to (35.6, 332.7), turned to 90 degrees
- moved J17 270.2 mm to (88.9, 275.6), turned to 90 degrees
- moved J18 254.9 mm to (35.6, 278.1), turned to 90 degrees
- moved J15 234.1 mm to (88.9, 248.9), turned to 90 degrees
- moved J16 221.3 mm to (35.6, 251.5), turned to 90 degrees
- moved B-CONNECTOR-14-LOWER-IN 210.7 mm to (104.1, 20.3), turned to 270 degrees
- moved B-CONNECTOR-14-LOWER-OUT 193.4 mm to (73.7, 19.1), flipped to the bottom, turned to 90 degrees
- moved A-CONNECTOR-14-LOWER-IN 133.1 mm to (44.5, 19.1), turned to 270 degrees
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Connections:
- removed net N$8: A-CONNECTOR-14-UPPER-IN.7, A-CONNECTOR-14-UPPER-OUT.7
- new net B-PASS1: B-CONNECTOR-14-LOWER-IN.3, B-CONNECTOR-14-LOWER-OUT.3
- new net B-PASS2: B-CONNECTOR-14-LOWER-IN.2, B-CONNECTOR-14-LOWER-OUT.2
- new net B-PASS3: B-CONNECTOR-14-LOWER-IN.1, B-CONNECTOR-14-LOWER-OUT.1
- new net N$5: A-CONNECTOR-14-UPPER-IN.11, A-CONNECTOR-14-UPPER-OUT.11
- net A1-B7: no longer B-CONNECTOR-14-LOWER-IN.1, B-CONNECTOR-14-LOWER-OUT.1
- net A19-B25: now also A-CONNECTOR-14-UPPER-IN.7, A-CONNECTOR-14-UPPER-OUT.7; no longer A-CONNECTOR-14-UPPER-IN.8, A-CONNECTOR-14-UPPER-OUT.8
- net A2-B8: no longer B-CONNECTOR-14-LOWER-IN.2, B-CONNECTOR-14-LOWER-OUT.2
- net A20-B26: now also A-CONNECTOR-14-UPPER-IN.8, A-CONNECTOR-14-UPPER-OUT.8; no longer A-CONNECTOR-14-UPPER-IN.9, A-CONNECTOR-14-UPPER-OUT.9
- net A21-B27: now also A-CONNECTOR-14-UPPER-IN.9, A-CONNECTOR-14-UPPER-OUT.9; no longer A-CONNECTOR-14-UPPER-IN.10, A-CONNECTOR-14-UPPER-OUT.10
- net A22-B28: now also A-CONNECTOR-14-UPPER-IN.10, A-CONNECTOR-14-UPPER-OUT.10; no longer A-CONNECTOR-14-UPPER-IN.11, A-CONNECTOR-14-UPPER-OUT.11
- net A3-B9: no longer B-CONNECTOR-14-LOWER-IN.3, B-CONNECTOR-14-LOWER-OUT.3
- net A4-B10: no longer A-CONNECTOR-14-UPPER-OUT.14
Routing:
- net A10-B16: track 0.00 -> 563.8 mm, vias 0 -> 5
- net A13-B19: track 0.00 -> 534.7 mm, vias 0 -> 9
- net A12-B18: track 0.00 -> 479.0 mm, vias 0 -> 3
- net A11-B17: track 0.00 -> 459.5 mm, vias 0 -> 4
- net A9-B15: track 0.00 -> 297.3 mm, vias 0 -> 1
- net A8-B14: track 0.00 -> 279.0 mm, vias 0 -> 1
- net A7-B13: track 0.00 -> 273.1 mm, vias 0 -> 3
- net A6-B12: track 0.00 -> 267.3 mm, vias 0 -> 1
- net A14-B20: track 0.00 -> 246.1 mm, vias 0 -> 5
- net A4-B10: track 0.00 -> 241.9 mm
- net A5-B11: track 0.00 -> 240.4 mm, vias 0 -> 1
- net A15-B21: track 0.00 -> 236.8 mm, vias 0 -> 4
- net A3-B9: track 0.00 -> 229.9 mm, vias 0 -> 2
- net A16-B22: track 0.00 -> 226.9 mm, vias 0 -> 6
- net A1-B7: track 0.00 -> 224.7 mm, vias 0 -> 2
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
Commit message: Update BMS Enerdel Adapter rev7.brd
Parts:
- moved J21 25.1 mm to (68.1, 315.0)
- moved J19 24.6 mm to (67.9, 289.3)
- moved J7 24.0 mm to (65.5, 135.5)
- moved J11 23.6 mm to (66.5, 186.7)
- moved J9 23.5 mm to (66.8, 159.6)
- moved J17 23.4 mm to (68.8, 263.5)
- moved J13 23.3 mm to (68.1, 211.8)
- moved J5 22.9 mm to (66.2, 111.3)
- moved J15 22.7 mm to (68.8, 238.3)
- moved J3 21.9 mm to (67.1, 86.6)
- moved J1 15.6 mm to (74.3, 55.4)
- moved J22 1.65 mm to (35.6, 331.1)
- moved J10 1.14 mm to (35.6, 170.1)
- moved J12 0.77 mm to (35.4, 197.6)
- moved J16 0.65 mm to (35.4, 250.8)
Routing:
- net A19-B25: track 185.9 -> 212.9 mm
- net A21-B27: track 199.2 -> 225.3 mm
- net A17-B23: track 194.4 -> 219.0 mm
- net A15-B21: track 236.8 -> 260.7 mm
- net A3-B9: track 229.9 -> 244.6 mm
- net A11-B17: track 459.5 -> 473.8 mm
- net A13-B19: track 534.7 -> 543.0 mm
- net A1-B7: track 224.7 -> 232.1 mm
- net A9-B15: track 297.3 -> 303.6 mm
- net A22-B28: track 182.7 -> 185.4 mm
- net A5-B11: track 240.4 -> 242.3 mm
- net A16-B22: track 226.9 -> 228.5 mm, vias 6 -> 5
- net A12-B18: track 479.0 -> 480.4 mm
- net A14-B20: track 246.1 -> 245.1 mm

Commit message: Update BMS Enerdel Adapter rev7.brd
Parts:
- moved J2 40.5 mm to (73.7, 76.1)
- moved J4 40.0 mm to (73.7, 101.0)
- moved J6 39.4 mm to (73.7, 125.6)
- moved J8 38.9 mm to (73.7, 150.2)
- moved J22 38.8 mm to (73.7, 323.6)
- moved J20 38.6 mm to (73.7, 298.3)
- moved J10 38.4 mm to (73.7, 174.8)
- moved J18 38.4 mm to (73.7, 273.6)
- moved J16 38.3 mm to (73.7, 248.9)
- moved J12 38.3 mm to (73.7, 199.4)
- moved J14 38.1 mm to (73.7, 224.3)
- moved J21 37.5 mm to (33.1, 301.4)
- moved J17 37.4 mm to (33.3, 252.0)
- moved J15 37.2 mm to (33.3, 227.3)
- moved J19 36.9 mm to (33.3, 276.6)
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Routing:
- net A10-B16: track 564.1 -> 454.6 mm, vias 5 -> 3
- net A12-B18: track 480.4 -> 371.5 mm, vias 3 -> 5
- net A13-B19: track 543.0 -> 437.5 mm, vias 9 -> 7
- net A11-B17: track 473.8 -> 370.9 mm, vias 4 -> 3
- net A21-B27: track 225.3 -> 153.8 mm, vias 3 -> 4
- net A9-B15: track 303.6 -> 234.6 mm, vias 1 -> 2
- net A19-B25: track 212.9 -> 150.4 mm, vias 3 -> 0
- net A7-B13: track 273.5 -> 212.3 mm, vias 3 -> 2
- net A15-B21: track 260.7 -> 201.6 mm
- net A20-B26: track 213.7 -> 156.4 mm
- net A3-B9: track 244.6 -> 187.4 mm, vias 2 -> 4
- net A6-B12: track 267.3 -> 210.6 mm
- net A5-B11: track 242.3 -> 187.8 mm, vias 1 -> 2
- net A1-B7: track 232.1 -> 178.0 mm, vias 2 -> 3
- net A18-B24: track 194.1 -> 145.0 mm, vias 2 -> 3
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Other:
- board size 329.9 x 382.3 mm -> 88.3 x 334 mm

Commit message: Matched enerdel holes to AMS holes
Parts:
- moved A-CONNECTOR-14-UPPER-OUT 416.9 mm to (-8.38, -78.2), turned to 0 degrees
- moved A-CONNECTOR-14-UPPER-IN 396.6 mm to (-8.00, -56.3), turned to 0 degrees
- moved B-CONNECTOR-14-UPPER-OUT 379.3 mm to (-10.9, -31.2), turned to 0 degrees
- moved J21 364.8 mm to (28.1, -63.4), turned to 180 degrees
- moved B-CONNECTOR-14-UPPER-IN 361.7 mm to (-10.9, -7.11), turned to 0 degrees
- moved J22 353.0 mm to (5.84, -22.9), turned to 180 degrees
- moved J19 340.4 mm to (52.8, -63.2), turned to 180 degrees
- moved J20 324.0 mm to (31.1, -22.9), turned to 180 degrees
- moved J17 318.3 mm to (77.5, -63.2), turned to 180 degrees
- moved J15 298.6 mm to (102.1, -63.2), turned to 180 degrees
- moved A-CONNECTOR-14-LOWER-OUT 298.3 mm to (291.1, -79.5), turned to 0 degrees
- moved J18 297.0 mm to (55.9, -22.9), turned to 180 degrees
- moved J13 281.9 mm to (126.7, -63.2), turned to 180 degrees
- moved J16 271.9 mm to (80.5, -22.9), turned to 180 degrees
- moved A-CONNECTOR-14-LOWER-IN 269.4 mm to (290.8, -57.4), turned to 0 degrees
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Other:
- board size 88.3 x 334 mm -> 342.9 x 87.6 mm

Commit message: Finished board
Parts:
- added U$1, U$3, U$4, U$5: (no value), HyTechAesthetics:HV_0.50"
- added U$2: (no value), HyTechAesthetics:LOGO_HYTECH_1.0"
Routing:
- net A5-B11: track 187.8 -> 197.1 mm, vias 2 -> 3
- net A3-B9: track 187.4 -> 188.5 mm
- net A4-B10: track 205.2 -> 206.1 mm
- net A21-B27: track 153.8 -> 154.7 mm
- net A13-B19: track 437.5 -> 436.6 mm
- net A2-B8: track 211.4 -> 212.0 mm
Other:
- board text added: "DANGER HIGH VOLTAGE"
- board text added: "Enerdel Adapter Rev 7 Designed by Stephen Noh"
- board text added: "Mode A"
- board text added: "Mode B"
- board text added: "Warning: DO NOT MIX Mode A and Mode B! Use only one mode at a time."

Commit message: final changes and order files
Parts:
- U$2: device HyTechAesthetics:LOGO_HYTECH_1.0" -> HyTechAesthetics:HV_0.50"
- U$5: device HyTechAesthetics:HV_0.50" -> HyTechAesthetics:LOGO_HYTECH_1.0"
- moved U$4 271.1 mm to (265.7, -81.6)
- moved J1 261.7 mm to (5.84, -22.9)
- moved U$3 260.1 mm to (5.64, -81.2)
- moved J22 246.5 mm to (249.0, -63.2)
- moved U$2 232.9 mm to (265.7, -9.68)
- moved U$5 232.9 mm to (44.9, -83.6)
- moved J2 222.2 mm to (31.1, -22.9)
- moved J21 197.4 mm to (225.4, -63.2)
- moved J3 197.3 mm to (55.9, -22.9)
- moved J20 174.4 mm to (200.8, -63.2)
- moved J4 148.0 mm to (80.5, -22.9)
- moved J12 137.5 mm to (267.6, -22.9)
- moved J5 126.9 mm to (105.2, -22.9)
- moved J19 123.2 mm to (176.0, -63.2)
- moved J11 109.7 mm to (253.4, -22.9)
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Connections:
- net A1-B7: now also J12.1; no longer J1.1
- net A10-B16: now also J7.1; no longer J10.1
- net A11-B17: now also J18.1; no longer J11.1
- net A12-B18: now also J6.1; no longer J12.1
- net A13-B19: now also J17.1; no longer J13.1
- net A14-B20: now also J5.1; no longer J14.1
- net A15-B21: now also J16.1; no longer J15.1
- net A16-B22: now also J4.1; no longer J16.1
- net A17-B23: now also J15.1; no longer J17.1
- net A18-B24: now also J3.1; no longer J18.1
- net A19-B25: now also J14.1; no longer J19.1
- net A2-B8: now also J11.1; no longer J2.1
- net A20-B26: now also J2.1; no longer J20.1
- net A21-B27: now also J13.1; no longer J21.1
- net A22-B28: now also J1.1; no longer J22.1
- net A3-B9: now also J22.1; no longer J3.1
- net A4-B10: now also J10.1; no longer J4.1
- net A5-B11: now also J21.1; no longer J5.1
- net A6-B12: now also J9.1; no longer J6.1
- net A7-B13: now also J20.1; no longer J7.1
- net A9-B15: now also J19.1; no longer J9.1
