File: EAGLE Board Designs/AMS/AMS Enerdel Adapter/BMS Enerdel Adapter rev8.sch (EAGLE design)
At the start: 48 parts, among them J1 CONNECTOR-1_5222_, J10 CONNECTOR-1_5222_, J11 CONNECTOR-1_5222_, J12 CONNECTOR-1_5222_, J13 CONNECTOR-1_5222_, J14 CONNECTOR-1_5222_, J15 CONNECTOR-1_5222_, J16 CONNECTOR-1_5222_, J17 CONNECTOR-1_5222_, J18 CONNECTOR-1_5222_, J19 CONNECTOR-1_5222_, J2 CONNECTOR-1_5222_, J20 CONNECTOR-1_5222_, J21 CONNECTOR-1_5222_, J22 CONNECTOR-1_5222_, J3 CONNECTOR-1_5222_, J4 CONNECTOR-1_5222_, J5 CONNECTOR-1_5222_, J6 CONNECTOR-1_5222_, J7 CONNECTOR-1_5222_, J8 CONNECTOR-1_5222_, J9 CONNECTOR-1_5222_

Commit message: some changes
Parts:
- A-CONNECTOR-14-LOWER-IN, A-CONNECTOR-14-LOWER-OUT: MPN (none) -> 39-28-1143
- F1, F10, F11, F12, F13, F14, F15, F16, F17, F18, F19, F2, F20, F21, F22, F3, F4, F5, F6, F7, F8, F9: value FUSE__.8 -> FUSE_MST_250_.8; device HyTechDevices:FUSE__.8 -> HyTechDevices:FUSE_MST_250_.8
Changed lines of the file:
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@@
 <part name="J22" library="HyTechDevices" deviceset="CONNECTOR-1_?_*" device="5222"/>
 <part name="J1" library="HyTechDevices" deviceset="CONNECTOR-1_?_*" device="5222"/>
-<part name="A-CONNECTOR-14-LOWER-IN" library="HyTechDevices" deviceset="CONNECTOR-14_?_*" device="MINIFIT"/>
-<part name="A-CONNECTOR-14-LOWER-OUT" library="HyTechDevices" deviceset="CONNECTOR-14_?_*" device="MINIFIT"/>
+<part name="A-CONNECTOR-14-LOWER-IN" library="HyTechDevices" deviceset="CONNECTOR-14_?_*" device="MINIFIT">
+<attribute name="MPN" value="
+39-28-1143"/>
+</part>
+<part name="A-CONNECTOR-14-LOWER-OUT" library="HyTechDevices" deviceset="CONNECTOR-14_?_*" device="MINIFIT">
+<attribute name="MPN" value="
+39-28-1143"/>
+</part>
 <part name="A-CONNECTOR-14-UPPER-IN" library="HyTechDevices" deviceset="CONNECTOR-14_?_*" device="NANOFIT"/>
 <part name="A-CONNECTOR-14-UPPER-OUT" library="HyTechDevices" deviceset="CONNECTOR-14_?_*" device="NANOFIT"/>
-<part name="F4" library="HyTechDevices" deviceset="FUSE_?_*" device="" technology=".8" value="FUSE__.8"/>
-<part name="F5" library="HyTechDevices" deviceset="FUSE_?_*" device="" technology=".8" value="FUSE__.8"/>
-<part name="F19" library="HyTechDevices" deviceset="FUSE_?_*" device="" technology=".8" value="FUSE__.8"/>
-<part name="F8" library="HyTechDevices" deviceset="FUSE_?_*" device="" technology=".8" value="FUSE__.8"/>
-<part name="F17" library="HyTechDevices" deviceset="FUSE_?_*" device="" technology=".8" value="FUSE__.8"/>
-<part name="F13" library="HyTechDevices" deviceset="FUSE_?_*" device="" technology=".8" value="FUSE__.8"/>
-<part name="F14" library="HyTechDevices" deviceset="FUSE_?_*" device="" technology=".8" value="FUSE__.8"/>
-<part name="F2" library="HyTechDevices" deviceset="FUSE_?_*" device="" technology=".8" value="FUSE__.8"/>
-<part name="F21" library="HyTechDevices" deviceset="FUSE_?_*" device="" technology=".8" value="FUSE__.8"/>
-<part name="F7" library="HyTechDevices" deviceset="FUSE_?_*" device="" technology=".8" value="FUSE__.8"/>
-<part name="F16" library="HyTechDevices" deviceset="FUSE_?_*" device="" technology=".8" value="FUSE__.8"/>
-<part name="F11" library="HyTechDevices" deviceset="FUSE_?_*" device="" technology=".8" value="FUSE__.8"/>
-<part name="F12" library="HyTechDevices" deviceset="FUSE_?_*" device="" technology=".8" value="FUSE__.8"/>
-<part name="F9" library="HyTechDevices" deviceset="FUSE_?_*" device="" technology=".8" value="FUSE__.8"/>
-<part name="F18" library="HyTechDevices" deviceset="FUSE_?_*" device="" technology=".8" value="FUSE__.8"/>
-<part name="F3" library="HyTechDevices" deviceset="FUSE_?_*" device="" technology=".8" value="FUSE__.8"/>
-<part name="F20" library="HyTechDevices" deviceset="FUSE_?_*" device="" technology=".8" value="FUSE__.8"/>
-<part name="F1" library="HyTechDevices" deviceset="FUSE_?_*" device="" technology=".8" value="FUSE__.8"/>
-<part name="F22" library="HyTechDevices" deviceset="FUSE_?_*" device="" technology=".8" value="FUSE__.8"/>
-<part name="F10" library="HyTechDevices" deviceset="FUSE_?_*" device="" technology=".8" value="FUSE__.8"/>
-<part name="F15" library="HyTechDevices" deviceset="FUSE_?_*" device="" technology=".8" value="FUSE__.8"/>
-<part name="F6" library="HyTechDevices" deviceset="FUSE_?_*" device="" technology=".8" value="FUSE__.8"/>
+<part name="F4" library="HyTechDevices" deviceset="FUSE_?_*" device="MST_250" technology=".8" value="FUSE_MST_250_.8"/>
+<part name="F5" library="HyTechDevices" deviceset="FUSE_?_*" device="MST_250" technology=".8" value="FUSE_MST_250_.8"/>
+<part name="F19" library="HyTechDevices" deviceset="FUSE_?_*" device="MST_250" technology=".8" value="FUSE_MST_250_.8"/>
+<part name="F8" library="HyTechDevices" deviceset="FUSE_?_*" device="MST_250" technology=".8" value="FUSE_MST_250_.8"/>
+<part name="F17" library="HyTechDevices" deviceset="FUSE_?_*" device="MST_250" technology=".8" value="FUSE_MST_250_.8"/>
+<part name="F13" library="HyTechDevices" deviceset="FUSE_?_*" device="MST_250" technology=".8" value="FUSE_MST_250_.8"/>
+<part name="F14" library="HyTechDevices" deviceset="FUSE_?_*" device="MST_250" technology=".8" value="FUSE_MST_250_.8"/>
+<part name="F2" library="HyTechDevices" deviceset="FUSE_?_*" device="MST_250" technology=".8" value="FUSE_MST_250_.8"/>
+<part name="F21" library="HyTechDevices" deviceset="FUSE_?_*" device="MST_250" technology=".8" value="FUSE_MST_250_.8"/>
+<part name="F7" library="HyTechDevices" deviceset="FUSE_?_*" device="MST_250" technology=".8" value="FUSE_MST_250_.8"/>
+<part name="F16" library="HyTechDevices" deviceset="FUSE_?_*" device="MST_250" technology=".8" value="FUSE_MST_250_.8"/>
+<part name="F11" library="HyTechDevices" deviceset="FUSE_?_*" device="MST_250" technology=".8" value="FUSE_MST_250_.8"/>
+<part name="F12" library="HyTechDevices" deviceset="FUSE_?_*" device="MST_250" technology=".8" value="FUSE_MST_250_.8"/>
+<part name="F9" library="HyTechDevices" deviceset="FUSE_?_*" device="MST_250" technology=".8" value="FUSE_MST_250_.8"/>
+<part name="F18" library="HyTechDevices" deviceset="FUSE_?_*" device="MST_250" technology=".8" value="FUSE_MST_250_.8"/>
+<part name="F3" library="HyTechDevices" deviceset="FUSE_?_*" device="MST_250" technology=".8" value="FUSE_MST_250_.8"/>
+<part name="F20" library="HyTechDevices" deviceset="FUSE_?_*" device="MST_250" technology=".8" value="FUSE_MST_250_.8"/>
+<part name="F1" library="HyTechDevices" deviceset="FUSE_?_*" device="MST_250" technology=".8" value="FUSE_MST_250_.8"/>
+<part name="F22" library="HyTechDevices" deviceset="FUSE_?_*" device="MST_250" technology=".8" value="FUSE_MST_250_.8"/>
+<part name="F10" library="HyTechDevices" deviceset="FUSE_?_*" device="MST_250" technology=".8" value="FUSE_MST_250_.8"/>
+<part name="F15" library="HyTechDevices" deviceset="FUSE_?_*" device="MST_250" technology=".8" value="FUSE_MST_250_.8"/>
+<part name="F6" library="HyTechDevices" deviceset="FUSE_?_*" device="MST_250" technology=".8" value="FUSE_MST_250_.8"/>
 </parts>
 <sheets>
@@
 <instance part="A-CONNECTOR-14-LOWER-IN" gate="G$1" x="142.24" y="142.24" smashed="yes" rot="R180">
 <attribute name="NAME" x="134.62" y="141.478" size="1.27" layer="95" rot="R180" align="bottom-right"/>
+<attribute name="MPN" x="142.24" y="142.24" size="1.778" layer="96" rot="R180"/>
 </instance>
 <instance part="A-CONNECTOR-14-LOWER-OUT" gate="G$1" x="101.6" y="142.24" smashed="yes" rot="MR180">
 <attribute name="NAME" x="109.22" y="141.478" size="1.27" layer="95" rot="MR180" align="bottom-right"/>
+<attribute name="MPN" x="101.6" y="142.24" size="1.778" layer="96" rot="MR180"/>
 </instance>
 <instance part="A-CONNECTOR-14-UPPER-IN" gate="G$1" x="63.5" y="142.24" smashed="yes" rot="R180">

Commit message: final changes and order files
Parts:
- A-CONNECTOR-14-LOWER-IN, A-CONNECTOR-14-LOWER-OUT: MPN 39-28-1143 -> 39-28-1143
- A-CONNECTOR-14-UPPER-IN, A-CONNECTOR-14-UPPER-OUT: MPN (none) -> 105310-1114
Connections:
- net N$10: now also J20.1; no longer J19.1
- net N$12: now also J19.1; no longer J18.1
- net N$14: now also J18.1; no longer J17.1
- net N$16: now also J13.1; no longer J22.1
- net N$18: now also J14.1; no longer J13.1
- net N$20: now also J15.1; no longer J14.1
- net N$22: now also J16.1; no longer J15.1
- net N$25: now also J17.1; no longer J16.1
- net N$3: now also J22.1; no longer J21.1
- net N$8: now also J21.1; no longer J20.1
Other:
- note removed: "B Mode"
- moved on the sheet: J13, J14, J15, J16, J17, J18, J19, J20, J21, J22
