File: External Diagrams/External Diagram FSAE 2022.sch (EAGLE design)
At the start: 100 parts, among them J1 CONNECTOR-22_SOURIAU_, J2 CONNECTOR-4_, J3 RING_TERMINAL_

Commit message: more rear diagram
Parts:
- removed D1, D2: DIODE_LED, HyTechSymbolsTemp:DIODE_LED
- removed DCDC_OUT_2: 39-01-2045, HyTechSymbols:M04
- removed POWER_ON_BTN: SWITCH_SPST_MOM, HyTechSymbols:SWITCH_SPST_MOM
Connections:
- removed net 12V_AFTER_LEFT_BRB: DCDC_CONTROL_IN_2.2
- removed net GND_DCDC_1: DCDC_OUT_2.1
- removed net GND_LEFT_PANEL: D2.C
- removed net N$54: DCDC_CONTROL_IN_2.1, POWER_ON_BTN.S
- net 12V_ACCUM: now also A1.M1-KL_30_BATT
- net 12V_DCDC_1: now also DCDC_12V_IN_2.1; no longer DCDC_12V_IN_2.3, DCDC_12V_IN_2.4, DCDC_OUT_2.3
- net 12V_DCDC_2: no longer DCDC_12V_IN_2.1, DCDC_OUT_2.4
- net 12V_MAIN: now also DCDC_IO_2.3, DCDC_IO_2.4; no longer A1.M1-KL_30_BATT, D1.A, D2.A, DCDC_IO_2.1, DCDC_IO_2.2
- net BAT+: now also DCDC_IO_2.1, DCDC_IO_2.2; no longer DCDC_IO_2.3, DCDC_IO_2.4, POWER_ON_BTN.P
- net GND_DCDC_2: no longer DCDC_OUT_2.2
- net GND_POWER_SWITCHING: now also DCDC_CONTROL_IN_2.1; no longer DCDC_CONTROL_IN_2.3
- net GND_RIGHT_PANEL: no longer D1.C, RIGHT_REAR_BRB.S1
Other:
- note added: "USB"

Commit message: shutdown circuit
Parts:
- removed F2: 10A, HyTechSymbols:FUSE
- added D1, D2: DIODE_LED, HyTechSymbolsTemp:DIODE_LED
- added S1: SWITCH_SPST_, HyTechSymbols:SWITCH_SPST_
Connections:
- removed net 12VSUPPLY_BRB: FIREWALL_3.1, FIREWALL_4.1, LEFT_REAR_BRB.O1, MAIN_SEC_1.1, MAIN_SEC_2.1
- removed net 12VSUPPLY_COOLING_UNSWITCHED: LEFT_REAR_BRB.P, RIGHT_REAR_BRB.O
- removed net 12VSUPPLY_UNSWITCHED: LEFT_REAR_BRB.P1, RIGHT_REAR_BRB.O1
- removed net N$74: F2.1, F3.1, GLVMS.S, MEASURE_12V.1
- new net 12V_SUPPLY: F3.2, FIREWALL_3.1, FIREWALL_4.1, MAIN_SEC_1.1, MAIN_SEC_2.1
- new net GND_LEFT_PANEL: D1.C
- new net N$17: D2.A, RIGHT_REAR_BRB.P1
- new net SHUTDOWN_L: A1.J3-HVP_IN, HVD_INTERLOCK.O
- new net SHUTDOWN_M: A1.J4-HVP_OUT, TSMS.P
- new net SHUTDOWN_N: TSMS.O
- new net START: DCDC_CONTROL_IN_2.3, S1.S
- net 12VSUPPLY_COOLING_PUMP_1: no longer LEFT_REAR_BRB.O
- net 12V_ACCUM: now also LEFT_REAR_BRB.P1, RIGHT_REAR_BRB.O1
- net BAT+: now also S1.P
- net GND_RIGHT_PANEL: now also D2.C
- net N$16: now also F3.1, GLVMS.S, MEASURE_12V.1; no longer F3.2, RIGHT_REAR_BRB.P
- net N$7: now also D1.A, LEFT_REAR_BRB.O1; no longer F2.2, RIGHT_REAR_BRB.P1
- net SHUTDOWN_H: no longer FIREWALL_1.9, FIREWALL_2.9, TSMS.P
- net SHUTDOWN_I: now also FIREWALL_1.9, FIREWALL_2.9, LEFT_REAR_BRB.P; no longer TSMS.S
- net SHUTDOWN_J: now also LEFT_REAR_BRB.O, RIGHT_REAR_BRB.O; no longer HVD_INTERLOCK.P
- net SHUTDOWN_K: now also HVD_INTERLOCK.P, RIGHT_REAR_BRB.P; no longer HVD_INTERLOCK.S
Other:
- note added: "START_BUTTON"
- moved on the sheet: F3, GLVMS, HVD_INTERLOCK, LEFT_REAR_BRB, MAINTENANCE, MEASURE_12V, MEASURE_GND, RIGHT_REAR_BRB, TSMS

Commit message: accum work
Parts:
- removed ACCUM_2: 8STA01035PN, HyTechSymbols:M13
- removed DCDC_OUT_1: 87427-0444, HyTechSymbols:M04
- removed DISCHARGE: (no value), HyTechDevices:RESISTOR10W
- removed FUSE9: 20A, HyTechSymbols:FUSE
- removed HVP_INTERLOCK: SWITCH_SPST, HyTechSymbols:SWITCH_SPST
- removed INDICATOR: INDICATOR, HyTechSymbols:LED
- removed PCB_F1, PCB_F2: 1A, HyTechSymbols:FUSE
- removed U$3: SMART_PRECHARGER, HyTechSymbols:SMART_PRECHARGER
- added J4: CONNECTOR-22_SOURIAU_, HyTechDevicesTemp:CONNECTOR-22_SOURIAU_
Connections:
- net IMD_SUPPLY renamed N$98
- removed net 60V_THRESHOLD: ACCUM_2.1
- removed net BMS_OK: ACCUM_2.4
- removed net CHARGE_ENABLE: ACCUM_2.2
- removed net HV+FUSED: PCB_F1.1
- removed net HV-FUSED: PCB_F2.1
- removed net IMD_GND: U$2.P1-GND, U$2.P3-GND, U$2.P4-GND
- removed net IMD_HV+: U$2.XLA+(HV+)
- removed net IMD_HV-: U$2.XLA-(HV-)
- removed net N$12: FUSE9.2, U$8.+OUT
- removed net N$13: DCDC_OUT_1.3, DCDC_OUT_1.4, FUSE9.1
- removed net N$14: DCDC_OUT_1.1, DCDC_OUT_1.2, U$8.-OUT
- removed net N$42: U$3.CTCS+
- removed net N$51: PCB_F1.2
- removed net N$52: PCB_F2.2
- removed net N$60: AIR2.P, U$3.CTCS-
- removed net SHUTDOWN_K_OUT: AIR1.1, U$3.12V
- new net N$100: U$2.P4-GND
- new net N$101: U$2.P5-PWM-HIGH
- new net N$102: U$2.P8-OKHS
- new net N$103: AIR1.2
- new net N$54: J4.9
- new net N$74: J4.11
- new net N$83: J4.7
- new net N$84: J4.8
- new net N$85: AIR1.1
- new net N$86: J4.16
- new net N$87: J4.17
- new net N$88: J4.18
- new net N$89: J4.19
- new net N$90: J4.22
- new net N$91: J4.21
- new net N$92: J4.20
- new net N$97: U$2.P1-GND
- new net N$99: U$2.P3-GND
- net 12V_ACCUM: no longer ACCUM_2.7
- net CANH_ACCUM: no longer ACCUM_2.10
- net CANL_ACCUM: no longer ACCUM_2.9
- net GND: no longer ACCUM_2.13, AIR1.2, U$3.GND
- net GND_ACCUM: no longer ACCUM_2.8
- net IMD_OK: no longer ACCUM_2.5, U$2.P8-OKHS
- net N$24: now also J4.4; no longer DISCHARGE.1
- net N$25: now also J4.5; no longer DISCHARGE.2
- net N$45: no longer U$3.COIL-
- net N$58: now also J4.10; no longer INDICATOR.A
- net N$59: now also J4.6; no longer INDICATOR.C
- net N$72: no longer U$3.COIL+
- net SHUTDOWN_I: no longer ACCUM_2.6, HVP_INTERLOCK.P
- net SHUTDOWN_J: no longer HVP_INTERLOCK.S
- net SHUTDOWN_N: now also A1.M3-KL15_EN, J1.11
- net SIGNAL_CURRENT: no longer ACCUM_2.3
- net USB_D+: no longer ACCUM_2.11
- net USB_D-: no longer ACCUM_2.12
Other:
- moved on the sheet: BMS_CELL_1, BMS_THERM_1, TSMP+A, TSMP-A

Commit message: add glvms to psb
Connections:
- net 12V_SUPPLY: now also DCDC_CONTROL_IN_2.2
Changed lines of the file:
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@@
 <drawing>
 <settings>
-<setting alwaysvectorfont="no"/>
+<setting alwaysvectorfont="yes"/>
 <setting keepoldvectorfont="yes"/>
 <setting verticaltext="up"/>
@@
 <wire x1="147.32" y1="7.62" x2="160.02" y2="7.62" width="0.1524" layer="91"/>
 </segment>
-</net>
+<segment>
+<pinref part="DCDC_CONTROL_IN_2" gate="G$1" pin="2"/>
+<wire x1="40.64" y1="71.12" x2="86.36" y2="71.12" width="0.1524" layer="91"/>
+<label x="86.36" y="71.12" size="1.778" layer="95" rot="MR0"/>
+</segment>
+</net>

Commit message: changes
Connections:
- net 12V_MAIN: now also MEASURE_12V.1
- net N$16: no longer MEASURE_12V.1
Other:
- moved on the sheet: MEASURE_12V
Changed lines of the file:
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@@
 <drawing>
 <settings>
-<setting alwaysvectorfont="yes"/>
+<setting alwaysvectorfont="no"/>
 <setting keepoldvectorfont="yes"/>
 <setting verticaltext="up"/>
@@
 <attribute name="VALUE" x="108.204" y="27.432" size="1.27" layer="96"/>
 </instance>
-<instance part="MEASURE_12V" gate="G$1" x="109.22" y="25.4" smashed="yes">
-<attribute name="NAME" x="108.204" y="27.178" size="1.27" layer="95"/>
-<attribute name="VALUE" x="108.204" y="22.352" size="1.27" layer="96"/>
+<instance part="MEASURE_12V" gate="G$1" x="109.22" y="25.4" smashed="yes" rot="R180">
+<attribute name="NAME" x="120.396" y="28.702" size="1.27" layer="95" rot="R180"/>
+<attribute name="VALUE" x="110.236" y="28.448" size="1.27" layer="96" rot="R180"/>
 </instance>
 <instance part="TSMP-A" gate="G$1" x="144.78" y="215.9" smashed="yes" rot="MR270">
@@
 <net name="12V_MAIN" class="0">
 <segment>
-<wire x1="132.08" y1="30.48" x2="132.08" y2="15.24" width="0.1524" layer="91"/>
+<wire x1="132.08" y1="30.48" x2="132.08" y2="25.4" width="0.1524" layer="91"/>
 <pinref part="GLVMS" gate="SPST" pin="P"/>
 <label x="152.4" y="30.48" size="1.778" layer="95"/>
 <label x="213.36" y="30.48" size="1.778" layer="95"/>
+<wire x1="132.08" y1="25.4" x2="132.08" y2="15.24" width="0.1524" layer="91"/>
 <wire x1="261.62" y1="30.48" x2="132.08" y2="30.48" width="0.1524" layer="91"/>
+<pinref part="MEASURE_12V" gate="G$1" pin="1"/>
+<wire x1="111.76" y1="25.4" x2="132.08" y2="25.4" width="0.1524" layer="91"/>
+<junction x="132.08" y="25.4"/>
 </segment>
 <segment>
@@
 <net name="N$16" class="0">
 <segment>
-<pinref part="MEASURE_12V" gate="G$1" pin="1"/>
-<wire x1="106.68" y1="25.4" x2="101.6" y2="25.4" width="0.1524" layer="91"/>
-<wire x1="101.6" y1="25.4" x2="101.6" y2="17.78" width="0.1524" layer="91"/>
 <pinref part="GLVMS" gate="SPST" pin="S"/>
 <wire x1="121.92" y1="17.78" x2="101.6" y2="17.78" width="0.1524" layer="91"/>
-<junction x="101.6" y="17.78"/>
 <wire x1="101.6" y1="17.78" x2="101.6" y2="7.62" width="0.1524" layer="91"/>
 <pinref part="F3" gate="G$1" pin="1"/>

Commit message: finish front and panel
Parts:
- removed BMS_CELL_1, BMS_THERM_1: 200277-1202, HyTechSymbols:M02
- removed BMS_CELL_2, BMS_THERM_2: 105307-1202, HyTechSymbols:M02
- removed BRAKE_1: 8STA00835PN, HyTechSymbols:M06
- removed BRAKE_2: 8STA60835SN, HyTechSymbols:M06
- removed DASH_COMM_1: 105308-1206, HyTechSymbols:M06
- removed DASH_COMM_2: 105310-1306, HyTechSymbols:M06
- removed DASH_IN_1: 105308-1208, HyTechSymbols:M08
- removed DASH_IN_2: 105310-1308, HyTechSymbols:M08
- removed F1: 20A, HyTechSymbols:FUSE
- removed F3: 10A, HyTechSymbols:FUSE
- removed FUSE1, FUSE7: 1.25A, HyTechSymbols:FUSE
- removed FUSE10_1A: (no value), HyTechSymbols:FUSE
- removed HVD: Hirose EM30MSD, HyTechSymbols:M02
- removed PED_1: 8STA01035PN, HyTechSymbols:M13
- removed PED_2: 8STA61035SN, HyTechSymbols:M13
- removed RTDS: BUZZER, HyTechSymbols:BUZZER
- removed SMD2B: PCL01, HyTechSymbols:M02
- removed U$8: DC-DC_CONVERTER, HyTechSymbols:DC-DC_CONVERTER
- added BPSD-, BSPD+: (no value), HyTechSymbols:BANANA_JACK
- added DASH_IN_3, DASH_IN_4: 105308-1208, HyTechSymbols:M08
- added HVD1: Hirose EM30MSD, HyTechSymbols:M02
- added HVD_3, HVD_4: TE_HVP800, HyTechSymbols:M02
- added J10, J11, J12, J13, J14, J5, J6, J7, J8, J9: CONNECTOR-3_, HyTechSymbolsTemp:CONNECTOR-3_
- added J15, J16: CONNECTOR-6_NF_T_V_BLACK, HyTechDevices:CONNECTOR-6_NF_T_V_BLACK
- added SMD2: PCL01, HyTechSymbols:M02
Connections:
- net N$45 renamed PRECHARGE_OK
- net N$85 renamed SHDN
- removed net N$103: AIR1.2
- removed net N$2: FUSE1.1, U$8.+IN
- removed net N$35: BMS_CELL_1.2
- removed net N$38: FUSE7.1, U$8.-IN
- removed net N$44: DASH_IN_1.1, RTDS.1
- removed net N$46: DASH_IN_1.4, RTDS.2
- removed net N$5 (its old number): FUSE1.2
- removed net N$61: BMS_THERM_1.1
- removed net N$62: BMS_THERM_1.2
- removed net N$63: BMS_THERM_2.1, BMS_THERM_2.2
- removed net N$68: F1.1, GLV_BATT.+
- removed net N$72: AIR2.1
- removed net N$75: FUSE10_1A.2
- removed net N$76: FUSE10_1A.1
- removed net N$9: FUSE7.2
- removed net SSOK: DASH_COMM_1.3
- new net BPSD+: BSPD+.1, J1.3
- new net BSPD-: BPSD-.1, J1.2
- new net N$12: J5.1
- new net N$13: J5.2
- new net N$14: J5.3
- new net N$24: J4.3
- new net N$36: J9.1
- new net N$51: J9.2
- new net N$52: J9.3
- new net N$6: J4.13
- net 12VSUPPLY_COOLING_PUMP_1: no longer PUMP_1.1
- net 12V_ACCUM: now also PUMP_1.1
- net 12V_DASH: now also DASH_IN_4.1; no longer DASH_COMM_1.1
- net 12V_SUPPLY: now also GLVMS.S; no longer F3.2
- net 5V_ACCEL_1: now also J11.2; no longer PED_1.6, PED_2.6
- net 5V_ACCEL_2: now also J12.2; no longer PED_1.2, PED_2.2
- net 5V_BRAKE_1: now also J7.1; no longer BRAKE_1.2
- net 5V_BRAKE_2: now also J8.1; no longer BRAKE_1.5
- net BAT+: now also GLV_BATT.+; no longer F1.2
- net CANH_DASH: now also DASH_IN_4.4; no longer DASH_COMM_1.5
- net CANL_DASH: now also DASH_IN_4.3; no longer DASH_COMM_1.4
- net GND: now also AIR1.2, AIR2.1
- net GND_ACCEL_1: now also J11.1; no longer PED_1.5, PED_2.5
- net GND_ACCEL_2: no longer PED_1.1, PED_2.1
- net GND_BRAKE_1: now also J7.2; no longer BRAKE_1.1
- net GND_BRAKE_2: now also J12.1, J8.2; no longer BRAKE_1.6
- net GND_DASH: now also DASH_IN_4.8; no longer DASH_COMM_1.2
- net N$1: now also J16.5; no longer DASH_IN_1.6
- net N$10: now also J4.15; no longer BMS_CELL_2.1, BMS_CELL_2.2
- net N$11: now also J4.12; no longer BMS_CELL_1.1
- net N$15: now also DASH_IN_3.1; no longer DASH_COMM_2.1
- net N$16: now also J6.1; no longer F3.1, GLVMS.S
- net N$18: now also DASH_IN_3.3; no longer DASH_COMM_2.2
- net N$19: now also DASH_IN_3.4; no longer DASH_COMM_2.3
- net N$21: now also DASH_IN_3.5; no longer DASH_COMM_2.4
- net N$22: now also DASH_IN_3.6; no longer DASH_COMM_2.6
- net N$23: now also DASH_IN_3.7; no longer DASH_COMM_2.5
- net N$26: now also J4.14; no longer DASH_IN_2.1
- net N$27: now also J15.1; no longer DASH_IN_2.2
- net N$28: now also J15.2; no longer DASH_IN_2.3
- net N$29: now also J15.3; no longer DASH_IN_2.4
- net N$30: now also J15.4; no longer DASH_IN_2.5
- net N$31: now also J15.5; no longer DASH_IN_2.6
- net N$32: now also J15.6; no longer DASH_IN_2.7
- net N$33: now also J4.2; no longer DASH_IN_2.8
- net N$37: now also J6.2; no longer BRAKE_2.2
- net N$41: now also J16.4; no longer DASH_IN_1.5
- net N$43: now also J16.3; no longer DASH_IN_1.3
- net N$47: now also J16.1; no longer DASH_IN_1.8
- net N$48: now also J16.2; no longer DASH_IN_1.2
- net N$49: now also J16.6; no longer DASH_IN_1.7
- net N$50: now also J6.3; no longer BRAKE_2.1
- net N$53: now also J10.1; no longer BRAKE_2.3
- net N$55: now also J10.2; no longer BRAKE_2.5
- net N$56: now also J10.3; no longer BRAKE_2.6
- net N$57: now also DASH_IN_3.8; no longer BRAKE_2.4
- net SHUTDOWN_E: no longer PED_1.12, PED_2.12
- net SHUTDOWN_F: now also DASH_IN_4.7, J13.1, J14.1
- net SHUTDOWN_G: now also DASH_IN_4.6, J13.2, J14.2; no longer PED_1.13, PED_2.13
- net SHUTDOWN_H: now also DASH_IN_4.5; no longer DASH_COMM_1.6
- net SIGNAL_ACCEL_1: now also J11.3; no longer PED_1.3
- net SIGNAL_ACCEL_2: now also J12.3; no longer PED_1.4
- net SIGNAL_BRAKE_1: now also J7.3; no longer BRAKE_1.3, PED_2.4
- net SIGNAL_BRAKE_2: now also J8.3; no longer BRAKE_1.4, PED_2.3
Other:
- note added: "8STA60435PA"
- note added: "8STA60435PB"
- note added: "8STA60435PN"
- note added: "8STA60435SA"
- note added: "8STA60435SB"
- note added: "8STA60435SN"
- note added: "BRAKE_1"
- note added: "BRAKE_2"
- note added: "HyTech Racing 2022 FSAE Electrical Diagram"
- note added: "PEDAL_1"
- note added: "PEDAL_2"
- note added: "PEDAL_3"
- note removed: "HyTech Racing 2021 FSAE Electrical Diagram"
- note removed: "⬅ BMS Cell Test Port"
- note removed: "⬅ BMS Therm Test Port"
- moved on the sheet: AIR2, BOTS, FUSE, INERTIA_SWITCH, J1, J4, SEGMENT1, SEGMENT2, SEGMENT3, SEGMENT4, SMD1, SMD2A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

Commit message: accumulator
Parts:
- added FUSE1, FUSE2: 1.25A, HyTechSymbols:FUSE
- added INDICATOR: LED_0603_RED, HyTechDevices:LED_0603_RED
Connections:
- removed net N$39: TSMP_RES-.2
- removed net N$40: TSMP_RES+.2
- new net N$103: TSMP-A.1, TSMP_RES-.2
- new net N$61: FUSE2.2
- new net N$62: FUSE1.2
- new net N$63: FUSE2.1
- new net N$68: FUSE1.1
- new net N$72: U$2.XLA+(HV+)
- new net N$76: U$2.XLA-(HV-)
- new net N$79: TSMP_RES+.1
- new net N$85: TSMP_RES-.1
- new net N$94: TSMP+A.1, TSMP_RES+.2
- net N$20: now also INDICATOR.A; no longer TSMP-A.1, TSMP_RES-.1
- net N$34: now also INDICATOR.C; no longer TSMP+A.1, TSMP_RES+.1
Other:
- moved on the sheet: FUSE, TSMP+A, TSMP-A, TSMP_RES+, TSMP_RES-

Commit message: change radiator wiring
Connections:
- net 12V_ACCUM: no longer PUMP_1.1
- net 12V_MAIN: now also PUMP_1.1
- net FAN_1: now also FIREWALL_3.2, FIREWALL_4.2
- net GND_RADIATOR: no longer FIREWALL_3.2, FIREWALL_4.2
Other:
- note added: "GND_RADIATOR"
Changed lines of the file:
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@@
 <drawing>
 <settings>
-<setting alwaysvectorfont="yes"/>
+<setting alwaysvectorfont="no"/>
 <setting keepoldvectorfont="yes"/>
 <setting verticaltext="up"/>
@@
 <wire x1="210.82" y1="264.16" x2="198.12" y2="264.16" width="0.6096" layer="156"/>
 <wire x1="187.96" y1="264.16" x2="162.56" y2="264.16" width="0.6096" layer="156"/>
+<text x="43.18" y="17.78" size="1.778" layer="95">GND_RADIATOR</text>
 </plain>
 <moduleinsts>
@@
 </instances>
 <busses>
-<bus name="5V_ACCEL_1,5V_ACCEL_2,5V_BRAKE,5V_BRAKE_1,5V_BRAKE_2,12V_ACCUM,12V_ACCUM_MAINT,12V_AFTER_LEFT_BRB,12V_DASH,12V_DCDC_1,12V_DCDC_2,12V_MAIN,12V_MAINT,12V_MC,12V_SUPPLY,12VSUPPLY_COOLING_FAN_1,12VSUPPLY_COOLING_FAN_2,12VSUPPLY_COOLING_FAN_3,12VSUPPLY_COOLING_PUMP_1,12VSUPPLY_COOLING_UNSWITCHED,12VSUPPLY_UNSWITCHED,12V_TSAL,12V_WHEEL_SPEED_FRONT_LEFT,12V_WHEEL_SPEED_FRONT_RIGHT,12V_WHEEL_SPEED_REAR_LEFT,12V_WHEEL_SPEED_REAR_RIGHT,60V_THRESHOLD,60V_THRESHOLD_1,60V_THRESHOLD_2,AMS_OK,BAT+,BPSD+,BRAKE_LIGHT,BSPD-,CAN_ACCUM_SHIELD,CANH_ACCUM,CANH_DASH,CANH_FRONT,CANH_MAINT,CANH_MC,CANL_ACCUM,CANL_DASH,CANL_MAINT,CANL_MC,CHARGE_ENABLE,CUR_SENSE_5V,CUR_SENSE_CUR_SENSE,CUR_SENSE_GND,CUR_SENSE_REF,DASH_1,DASH_4,DASH_5,DASH_8,DASH_9,DASH_11,DASH_12,FAN_1,FAN_2,GND,GND_ACCEL_1,GND_ACCEL_2,GND_ACCUM,GND_AUX,GND_BR,GND_BRAKE,GND_BRAKE_1,GND_BRAKE_2,GND_BR_TS,GND_CHASSIS,GND_CURRENT,GND_DASH,GND_DCDC1,GND_DCDC_1,GND_DCDC_2,GND_DCDC2,GND_DCDC_4,GND_LEFT_PANEL,GND_MAIN_ECU,GND_MAINT,GND_MC,GND_POWER_SWITCHING,GND_RADIATOR,GND_RIGHT_PANEL,GND_SHIELD,GND_TSAL_GREEN,GND_TSAL_RED,HV+,HV-,HV+FUSED,HV-FUSED,IMD_GND,IMD_HV+,IMD_HV-,IMD_OK,IMD_SUPPLY,INVERTER_SUPPLY,ISOSPI_M,ISOSPI_P,LATCH_EXT_BTN,MC_MAINT_FAULT_INDIC,MC_MAINT_GND,MC_MAINT_PROG_ENA,MC_MAINT_RXD,MC_MAINT_TXD,MC_MAINT_XDCR_PWR,MOTOR_COS-,MOTOR_COS+,MOTOR_EXC-,MOTOR_EXC+,MOTOR_SHIELD,MOTOR_SIN-,MOTOR_SIN+,MOTOR_TEMP+,MOTOR_TEMP-,RET_FAN_1,SHUTDOWN_E,SHUTDOWN_F,SHUTDOWN_G,SHUTDOWN_H,SHUTDOWN_I,SHUTDOWN_J,SHUTDOWN_K,SHUTDOWN_K_OUT,SHUTDOWN_L,SHUTDOWN_M,SHUTDOWN_N,SIGNAL_ACCEL_1,SIGNAL_ACCEL_2,SIGNAL_BRAKE,SIGNAL_BRAKE_1,SIGNAL_BRAKE_2,SIGNAL_CURRENT,SSOK,START,USB_D-,USB_D+,USB_GND,USB_VCC,WHEEL_SPEED_2,WHEEL_SPEED_3,WHEEL_SPEED_4,WHEEL_SPEED_FRONT_LEFT,WHEEL_SPEED_FRONT_RIGHT,WHEEL_SPEED_REAR_LEFT,WHEEL_SPEED_REAR_RIGHT">
+<bus name="5V_ACCEL_1,5V_ACCEL_2,5V_BRAKE,5V_BRAKE_1,5V_BRAKE_2,12V_ACCUM_MAINT,12V_AFTER_LEFT_BRB,12V_DASH,12V_DCDC_1,12V_DCDC_2,12V_MAIN,12V_MAINT,12V_MC,12V_SUPPLY,12VSUPPLY_COOLING_FAN_1,12VSUPPLY_COOLING_FAN_2,12VSUPPLY_COOLING_FAN_3,12VSUPPLY_COOLING_PUMP_1,12VSUPPLY_COOLING_UNSWITCHED,12VSUPPLY_UNSWITCHED,12V_TSAL,12V_WHEEL_SPEED_FRONT_LEFT,12V_WHEEL_SPEED_FRONT_RIGHT,12V_WHEEL_SPEED_REAR_LEFT,12V_WHEEL_SPEED_REAR_RIGHT,60V_THRESHOLD,60V_THRESHOLD_1,60V_THRESHOLD_2,AMS_OK,BAT+,BPSD+,BRAKE_LIGHT,BSPD-,CAN_ACCUM_SHIELD,CANH_ACCUM,CANH_DASH,CANH_FRONT,CANH_MAINT,CANH_MC,CANL_ACCUM,CANL_DASH,CANL_MAINT,CANL_MC,CHARGE_ENABLE,CUR_SENSE_5V,CUR_SENSE_CUR_SENSE,CUR_SENSE_GND,CUR_SENSE_REF,DASH_1,DASH_4,DASH_5,DASH_8,DASH_9,DASH_11,DASH_12,FAN_1,FAN_2,GND,GND_ACCEL_1,GND_ACCEL_2,GND_ACCUM,GND_AUX,GND_BR,GND_BRAKE,GND_BRAKE_1,GND_BRAKE_2,GND_BR_TS,GND_CHASSIS,GND_CURRENT,GND_DASH,GND_DCDC1,GND_DCDC_1,GND_DCDC_2,GND_DCDC2,GND_DCDC_4,GND_LEFT_PANEL,GND_MAIN_ECU,GND_MAINT,GND_MC,GND_POWER_SWITCHING,GND_RIGHT_PANEL,GND_SHIELD,GND_TSAL_GREEN,GND_TSAL_RED,HV+,HV-,HV+FUSED,HV-FUSED,IMD_GND,IMD_HV+,IMD_HV-,IMD_OK,IMD_SUPPLY,INVERTER_SUPPLY,ISOSPI_M,ISOSPI_P,LATCH_EXT_BTN,MC_MAINT_FAULT_INDIC,MC_MAINT_GND,MC_MAINT_PROG_ENA,MC_MAINT_RXD,MC_MAINT_TXD,MC_MAINT_XDCR_PWR,MOTOR_COS-,MOTOR_COS+,MOTOR_EXC-,MOTOR_EXC+,MOTOR_SHIELD,MOTOR_SIN-,MOTOR_SIN+,MOTOR_TEMP+,MOTOR_TEMP-,RET_FAN_1,SHUTDOWN_E,SHUTDOWN_F,SHUTDOWN_G,SHUTDOWN_H,SHUTDOWN_I,SHUTDOWN_J,SHUTDOWN_K,SHUTDOWN_K_OUT,SHUTDOWN_L,SHUTDOWN_M,SHUTDOWN_N,SIGNAL_ACCEL_1,SIGNAL_ACCEL_2,SIGNAL_BRAKE,SIGNAL_BRAKE_1,SIGNAL_BRAKE_2,SIGNAL_CURRENT,SSOK,START,USB_D-,USB_D+,USB_GND,USB_VCC,WHEEL_SPEED_2,WHEEL_SPEED_3,WHEEL_SPEED_4,WHEEL_SPEED_FRONT_LEFT,WHEEL_SPEED_FRONT_RIGHT,WHEEL_SPEED_REAR_LEFT,WHEEL_SPEED_REAR_RIGHT">
 <segment>
 <wire x1="627.38" y1="17.78" x2="627.38" y2="48.26" width="0.762" layer="92"/>
@@
 <label x="91.44" y="220.98" size="1.778" layer="95" rot="R90"/>
 </segment>
-<segment>
-<pinref part="PUMP_1" gate="G$1" pin="1"/>
-<wire x1="0" y1="60.96" x2="40.64" y2="60.96" width="0.1524" layer="91"/>
-<label x="2.54" y="60.96" size="1.778" layer="95"/>
-</segment>
 </net>
 <net name="GND_CURRENT" class="0">
@@
 <label x="322.58" y="38.1" size="1.778" layer="95"/>
 </segment>
+<segment>
+<pinref part="FIREWALL_3" gate="G$1" pin="2"/>
+<wire x1="363.22" y1="-10.16" x2="320.04" y2="-10.16" width="0.1524" layer="91"/>
+<label x="322.58" y="-10.16" size="1.778" layer="95"/>
+</segment>
+<segment>
+<pinref part="FIREWALL_4" gate="G$1" pin="2"/>
+<wire x1="434.34" y1="-10.16" x2="388.62" y2="-10.16" width="0.1524" layer="91"/>
+<label x="391.16" y="-10.16" size="1.778" layer="95"/>
+</segment>
 </net>
 <net name="N$27" class="0">
@@
 <pinref part="PUMP_2" gate="G$1" pin="2"/>
 </segment>
-<segment>
-<pinref part="FIREWALL_4" gate="G$1" pin="2"/>
-<wire x1="434.34" y1="-10.16" x2="388.62" y2="-10.16" width="0.1524" layer="91"/>
-<label x="391.16" y="-10.16" size="1.778" layer="95"/>
-</segment>
-<segment>
-<pinref part="FIREWALL_3" gate="G$1" pin="2"/>
-<wire x1="363.22" y1="-10.16" x2="320.04" y2="-10.16" width="0.1524" layer="91"/>
-<label x="322.58" y="-10.16" size="1.778" layer="95"/>
-</segment>
 </net>
 <net name="SHUTDOWN_I" class="0">
@@
 <wire x1="236.22" y1="66.04" x2="261.62" y2="66.04" width="0.1524" layer="91"/>
 </segment>
+<segment>
+<pinref part="PUMP_1" gate="G$1" pin="1"/>
+<wire x1="0" y1="60.96" x2="40.64" y2="60.96" width="0.1524" layer="91"/>
+<label x="2.54" y="60.96" size="1.778" layer="95"/>
+</segment>
 </net>
 <net name="GND_DCDC_2" class="0">
@@
 <wire x1="88.9" y1="15.24" x2="40.64" y2="15.24" width="0.1524" layer="91"/>
 <label x="43.18" y="15.24" size="1.778" layer="95"/>
+<wire x1="88.9" y1="15.24" x2="88.9" y2="17.78" width="0.1524" layer="91"/>
+<wire x1="88.9" y1="17.78" x2="40.64" y2="17.78" width="0.1524" layer="91"/>
 </segment>
 <segment>
